File: eagle/touch_glove/touch_glove.sch (EAGLE design)
At the start: 61 parts, among them P1 PELTIER, P2 PELTIER, P3 PELTIER, P4 PELTIER, P5 PELTIER, U2 DRV8837C, U3 DRV8837C, U4 DRV8837C, U5 DRV8837C, U6 DRV8837C

Commit message: Modified gitignore.  Tons of progress on PCB for Touch Glove
Parts:
- removed F1: FSR, MrSwirlyEyes:FSR_FORCE-SENSATIVE-RESISTOR_PRESS-SENSOR
- added A1: ANTENNASMD5, lib_kenmei:ANTENNASMD5
- added B1: 748421245, lib_kenmei:BALUN0805
- added C23, C27, C28, C29: 10uF/25V, MrSwirlyEyes:CAP_CERAMIC_SMD-805_10UF-25V-10%
- added C24, C25, C26, C30, C31, C32, C33, C34, C35, C37, C39, C46: 0.1uF/50V, MrSwirlyEyes:CAP_CERAMIC_SMD-805_0.1UF-50V-10%
- added C36, C38, C40, C41, C47: 1uF/25V, MrSwirlyEyes:CAP_CERAMIC_SMD-805-1UF-25V-10%
- added C42, C43: 12pF/250V, MrSwirlyEyes:CAP_CERAMIC_SMD-805_12PF-250V-5%
- added C44: 22PF/250V, MrSwirlyEyes:CAP_CERAMIC_SMD-805_22PF-250V-5%
- added C45: 0.75PF/100V, MrSwirlyEyes:CAP_CERAMIC_SMD-805-0.75PF-100V-33%
- added FLEX1, FLEX2, FLEX3, FLEX4, FLEX5: 10K, MrSwirlyEyes:FLEX-SENSOR10K_2.2IN
- added R12, R13: 4.7K, MrSwirlyEyes:RESISTORSMD-0805_1/8W_4.7K_5%
- added R14, R16, R18, R20, R22, R24, R26, R28, R30, R32, R34, R35, R36, R37, R38: 10KΩ, MrSwirlyEyes:RESISTORSMD-0805_1/8W_10K_5%
- added R15, R17, R19, R21, R23, R25, R27, R29, R31, R33: 100Ω, MrSwirlyEyes:RESISTORSMD-0805_1/8W_100_5%
- added U1: DRV8837C, MrSwirlyEyes:DRV8837C_H-BRIDGE_1A_WSON-8-PADDRV8837C_1A
- added Y1: 16MHz, MrSwirlyEyes:CRYSTAL_ABM3B_16MHZ_18PF
- C1, C11, C14, C15, C18: value 0.1uF/50V -> 10uF/25V; device MrSwirlyEyes:CAPACITOR_CERAMIC_SMD-805_0.1UF-50V-10% -> MrSwirlyEyes:CAP_CERAMIC_SMD-805_10UF-25V-10%
- C10, C19, C22: value 100UF/16V -> 10uF/25V; device MrSwirlyEyes:CAPACITOR_POLARIZED_ALUM-ELECTROLYTIC_SMD_100UF-16V-20% -> MrSwirlyEyes:CAP_CERAMIC_SMD-805_10UF-25V-10%
- C12, C17, C20, C21, C3, C4, C5, C6, C7, C8, C9: device MrSwirlyEyes:CAPACITOR_CERAMIC_SMD-805_0.1UF-50V-10% -> MrSwirlyEyes:CAP_CERAMIC_SMD-805_0.1UF-50V-10%
- C13, C16: value 100UF/16V -> 0.1uF/50V; device MrSwirlyEyes:CAPACITOR_POLARIZED_ALUM-ELECTROLYTIC_SMD_100UF-16V-20% -> MrSwirlyEyes:CAP_CERAMIC_SMD-805_0.1UF-50V-10%
- C2: value 10uF/25V -> 0.1uF/50V; device MrSwirlyEyes:CAPACITOR_CERAMIC_SMD-805_10UF-25V-10% -> MrSwirlyEyes:CAP_CERAMIC_SMD-805_0.1UF-50V-10%
- D1, D2, D3, D4, D5: device MrSwirlyEyes:DIODE_SMD_GP_1A-50V-SOD123F -> MrSwirlyEyes:DIODE_GEN-PURPSMD_GP_1A-50V-SOD123F
- P1, P2, P3, P4, P5: device MrSwirlyEyes:PELTIER-CM23-1.9-05AC_1.9A-2.8V_8X6X2MM -> MrSwirlyEyes:PELTIER-TECNL1025T_1.8A-4.4V_L10.7-W8.8-H2
- R10, R6, R7, R8, R9: value 10KΩ -> 100Ω; device MrSwirlyEyes:RESISTORSMD-0805_1/8W_10K_5% -> MrSwirlyEyes:RESISTORSMD-0805_1/8W_100_5%
- U2, U3, U4, U5: device MrSwirlyEyes:DRV8837C_H-BRIDGE_1A_WSON-8-PAD -> MrSwirlyEyes:DRV8837C_H-BRIDGE_1A_WSON-8-PADDRV8837C_1A
- U6: value DRV8837C -> ATMEGA128RFA1; device MrSwirlyEyes:DRV8837C_H-BRIDGE_1A_WSON-8-PAD -> MrSwirlyEyes:ATMEGA128RFA1
Connections:
- new net A0: U6.PF0(ADC0)
- new net A1: U6.PF1(ADC1)
- new net A2: U6.PF2(ADC2/DIG2)
- new net A3: U6.PF3(ADC3/DIG4)
- new net A4: U6.PF4(ADC4/TCK)
- new net A5: U6.PF5(ADC5/TMS)
- new net A6: U6.PF6(ADC6/TDO)
- new net A7: U6.PF7(ADC7/TDI)
- new net C15: DEMUX.C15
- new net FSR_2: FLEX2.-, R34.2
- new net FSR_3: FLEX3.-, R35.2
- new net FSR_4: FLEX4.-, R36.2
- new net FSR_5: FLEX5.-, R37.2
- new net MISO: U6.PB3(MISO/PDO/PCINT3)
- new net MOSI: U6.PB2(MOSI/PDI/PCINT2)
- new net N$21: R9.2, VIBE_T4.G
- new net N$22: R10.2, VIBE_T5.G
- new net N$23: P5.HOT, U5.OUT1
- new net N$24: P5.COLD, U5.OUT2
- new net N$25: R27.2, U5.IN2
- new net N$26: R29.2, U5.IN1
- new net N$27: P4.HOT, U4.OUT1
- new net N$28: P4.COLD, U4.OUT2
- new net N$29: R31.2, U4.IN2
- new net N$30: C43.1, U6.XTAL1, Y1.2
- new net N$31: R33.2, U4.IN1
- new net N$32: B1.OUT2, U6.RFN
- new net N$33: B1.OUT1, U6.RFP
- new net N$34: B1.GND@2, C44.1
- new net N$35: C42.1, U6.XTAL2, Y1.1
- new net N$39: A1.SIGNAL, B1.IN, C45.1
- new net PB4: U6.PB4(OC2A/PCINT4)
- new net PB5: U6.PB5(OC1A/PCINT5)
- new net PB6: U6.PB6(OC1B/PCINT6)
- new net PB7: U6.PB7(OC0A/OC1C/PCINT7)
- new net PD4: U6.PD4(ICP1)
- new net PD5: U6.PD5(XCK1)
- new net PD6: U6.PD6(T1)
- new net PD7: U6.PD7(T0)
- new net PE2: U6.PE2(XCK0/AIN0)
- new net PE3: U6.PE3(OC3A/AIN1)
- new net PE4: U6.PE4(OC3B/INT4)
- new net PE5: U6.PE5(OC3C/INT5)
- new net PE6: U6.PE6(T3/INT6)
- new net PE7: U6.PE7(ICP3/INT7/CLKO)
- new net PG0: U6.PG0(DIG3)
- new net PG1: U6.PG1(DIG1)
- new net PG2: U6.PG2(AMR)
- new net PG3: U6.PG3(TOSC2)
- new net PG4: U6.PG4(TOSC1)
- new net PG5: U6.PG5(OC0B)
- new net RESET: R38.1, U6.RSTN
- new net RX0: U6.PE0(RXD0/PCINT8)
- new net RX1: U6.PD2(RXD1/INT2)
- new net SCK: U6.PB1(SCK/PCINT1)
- new net SS: U6.PB0(SSN/PCINT0)
- new net TX0: U6.PE1(TXD0)
- new net TX1: U6.PD3(TXD1/INT3)
- new net VM: C10.1, C13.1, C14.1, C17.1, C18.1, C21.1, C22.1, C26.1, C27.1, C9.1, U1.VM, U2.VM, U3.VM, U4.VM, U5.VM
- net FSR_1: now also FLEX1.-; no longer DEMUX.C15, F1.-
- net GND: now also B1.GND@5, C10.2, C13.2, C16.2, C19.2, C22.2, C23.2, C24.2, C25.2, C26.2, C27.2, C28.2, C29.2, C30.2, C31.2, C32.2, C33.2, C34.2, C35.2, C36.2, C37.2, C38.2, C39.2, C40.2, C41.2, C42.2, C43.2, C44.2, C45.2, C46.2, C47.2, R14.1, R16.1, R18.1, R20.1, R22.1, R24.1, R26.1, R28.1, R30.1, R32.1, R34.1, R35.1, R36.1, R37.1, U1.GND, U6.AVSS, U6.AVSS_RFN, U6.AVSS_RFP, U6.CLKI, U6.DVSS, U6.TST; no longer C10.K, C13.K, C16.K, C19.K, C22.K, U6.GND
- net N$1: now also P1.HOT, U1.OUT1; no longer P2.HOT, U3.OUT1
- net N$10: now also R17.2, U1.IN1; no longer R7.1
- net N$11: now also P2.HOT, U2.OUT1; no longer P3.HOT, U4.OUT1
- net N$12: now also P2.COLD, U2.OUT2; no longer P3.COLD, U4.OUT2
- net N$13: now also R19.2, U2.IN2; no longer P1.HOT, U2.OUT1
- net N$14: now also R21.2, U2.IN1; no longer P1.COLD, U2.OUT2
- net N$16: now also P3.HOT, U3.OUT1; no longer P4.HOT, U5.OUT1
- net N$18: now also P3.COLD, U3.OUT2; no longer P4.COLD, U5.OUT2
- net N$19: now also R23.2, U3.IN2; no longer P5.HOT, U6.OUT1
- net N$20: now also R25.2, U3.IN1; no longer P5.COLD, U6.OUT2
- net N$5: now also P1.COLD, U1.OUT2; no longer P2.COLD, U3.OUT2
- net N$6: now also R6.2, VIBE_T1.G; no longer R6.1
- net N$7: now also R7.2, VIBE_T2.G; no longer R10.1
- net N$8: now also R15.2, U1.IN2; no longer R9.1
- net N$9: now also R8.2, VIBE_T3.G; no longer R8.1
- net SCL: now also R13.1, U6.PD0(SCL/INT0)
- net SDA: now also R12.1, U6.PD1(SDA/INT1)
- net TEC_1_COLD: now also R26.2, R27.1; no longer U2.IN2
- net TEC_1_HOT: now also R28.2, R29.1; no longer U2.IN1
- net TEC_2_COLD: now also R22.2, R23.1; no longer U3.IN2
- net TEC_2_HOT: now also R24.2, R25.1; no longer U3.IN1
- net TEC_3_COLD: now also R18.2, R19.1; no longer U4.IN2
- net TEC_3_HOT: now also R20.2, R21.1; no longer U4.IN1
- net TEC_4_COLD: now also R14.2, R15.1; no longer U5.IN2
- net TEC_4_HOT: now also R16.2, R17.1; no longer U5.IN1
- net TEC_5_COLD: now also R30.2, R31.1; no longer U6.IN2
- net TEC_5_HOT: now also R32.2, R33.1; no longer U6.IN1
- net VCC: now also C16.1, C19.1, C23.1, C24.1, C25.1, C28.1, C29.1, C30.1, C31.1, C32.1, C33.1, C34.1, C35.1, C36.1, C37.1, C38.1, C39.1, C40.1, C41.1, C46.1, C47.1, FLEX1.+, FLEX2.+, FLEX3.+, FLEX4.+, FLEX5.+, R12.2, R13.2, R38.2, U1.NSLEEP, U1.VCC, U6.AREF, U6.AVDD, U6.DEVDD, U6.DVDD, U6.EVDD; no longer C10.A, C13.A, C14.1, C16.A, C17.1, C18.1, C19.A, C21.1, C22.A, C9.1, F1.+, U2.VM, U3.VM, U4.VM, U5.VM, U6.NSLEEP, U6.VCC, U6.VM
- net VIBE_1: now also R6.1; no longer R6.2, VIBE_T1.G
- net VIBE_2: now also R7.1; no longer R7.2, VIBE_T2.G
- net VIBE_3: now also R8.1; no longer R8.2, VIBE_T3.G
- net VIBE_4: now also R9.1; no longer R9.2, VIBE_T4.G
- net VIBE_5: now also R10.1; no longer R10.2, VIBE_T5.G
Other:
- note added: "47K?"
- note added: "ATMEGA128RFA1"
- note added: "FLEX/STRAIN SENSORS"
- note added: "IMU"
- note added: "Might add op amps"
- note added: "NC"
- note removed: "CHANGE TO VBATT or VM"
- moved on the sheet: C1, C11, C12, C14, C15, C17, C18, C2, C20, C21, C8, C9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

Commit message: Modified TMP36 temperature sensor library to work with DEMUX.  Added ATMEGA128RFA1 and LM9DS1 IMU to Touch Glove schematic
Parts:
- added C48: 0.22uF/50V, MrSwirlyEyes:CAP_CERAMIC_SMD-805_0.22UF-50V-10%
- added C49, C50: 10uF/25V, MrSwirlyEyes:CAP_CERAMIC_SMD-805_10UF-25V-10%
- added C51: 0.1uF/50V, MrSwirlyEyes:CAP_CERAMIC_SMD-805_0.1UF-50V-10%
- added IMU1: LM9DS1, lib_kenmei:LSM9DS1_IMU
Connections:
- new net N$36: C49.1, IMU1.CAP
- new net N$37: C48.1, IMU1.C1
- net GND: now also C48.2, C49.2, C50.2, C51.2, IMU1.GND@1, IMU1.GND@2, IMU1.RES@1, IMU1.RES@2, IMU1.RES@3, IMU1.RES@4, IMU1.RES@5
- net SCL: now also IMU1.SCL/SPC, R12.1; no longer R13.1
- net SDA: now also IMU1.SDA/SDI/SDO, R13.1; no longer R12.1
- net VCC: now also C50.1, C51.1, IMU1.VDD@1, IMU1.VDD@2, IMU1.VDDIO@1, IMU1.VDDIO@2
Other:
- note added: "IMU LM9DS1"
- note removed: "IMU"
- moved on the sheet: R12, R13

Commit message: Added FTDI programmer and AVR SPI bootloader pins to schematic
Parts:
- added C52, C53, C54, C55, C56, C62: 0.1uF/50V, MrSwirlyEyes:CAP_CERAMIC_SMD-805_0.1UF-50V-10%
- added C57, C58, C59, C60, C61: 10uF/25V, MrSwirlyEyes:CAP_CERAMIC_SMD-805_10UF-25V-10%
- added J1: (no value), MrSwirlyEyes:AVR_SPI_PRG_6NS
- added JP1: FTDIPTH-RA, MrSwirlyEyes:FTDIPTH-RA
Connections:
- net SS renamed SSN
- new net N$41: C62.1, JP1.2
- new net N$42: JP1.5
- net GND: now also C52.2, C53.2, C54.2, C55.2, C56.2, C57.2, C58.2, C59.2, C60.2, C61.2, J1.6, JP1.6
- net MISO: now also J1.1
- net MOSI: now also J1.4
- net RESET: now also C62.2, J1.5
- net RX0: now also JP1.4
- net SCK: now also J1.3
- net TX0: now also JP1.3
- net VCC: now also C52.1, C53.1, C54.1, C55.1, C56.1, C57.1, C58.1, C59.1, C60.1, C61.1, J1.2, JP1.1
Other:
- note added: "ACTUATORS"
- note added: "AVR ISP"
- note added: "CHECK THESE FOR ACCURACY"
- note added: "DEMULTIPLEXER"
- note added: "FLEX SENSORS"
- note added: "FTDI"
- note added: "Maybe one for palm?"
- note added: "POWER"
- note added: "PROGRAMMER"
- note added: "SENSORS"
- note removed: "DEMUX for STRAIN SENSORS"
- note removed: "FLEX/STRAIN SENSORS"
- moved on the sheet: A1, B1, C1, C2, C23, C24, C3, C30, C31, C32, C33, C34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
