File: eagle/touch_glove/touch_glove.sch (EAGLE design)
At the start: 139 parts, among them P1 PELTIER, P2 PELTIER, P3 PELTIER, P4 PELTIER, P5 PELTIER, U1 DRV8837C, U2 DRV8837C, U3 DRV8837C, U4 DRV8837C, U5 DRV8837C, U6 ATMEGA128RFA1, Y1 16MHz

Commit message: Changed power symbols for Glove
Parts:
- added BATT1: BATTERYPTH_HOLES, MrSwirlyEyes:BATTERYPTH_HOLES
- added C63, C64, C65, C66, C69, C70, C71: 10uF/25V, MrSwirlyEyes:CAP_CERAMIC_SMD-805_10UF-25V-10%
- added C67: 220uF/16V, MrSwirlyEyes:CAP_POLARIZED_ALUM-ELECTROLYTIC_SMD_220UF-16V-20%
- added C68, C74, C75, C76: 0.1uF/50V, MrSwirlyEyes:CAP_CERAMIC_SMD-805_0.1UF-50V-10%
- added C78: 100UF/16V, MrSwirlyEyes:CAP_POLARIZED_ALUM-ELECTROLYTIC_SMD_100UF-16V-20%
- added C79: 1uF/25V, MrSwirlyEyes:CAP_CERAMIC_SMD-805-1UF-25V-10%
- added D6, D7, D8: 1A/50V, MrSwirlyEyes:DIODE_GEN-PURPSMD_GP_1A-50V-SOD123F
- added L1, L2: 10uH, MrSwirlyEyes:INDUCTORSMD-805_10UH-0.5A-0.65OHM-10%
- added SW1: 5A/28V, MrSwirlyEyes:SWITCH_SPDT5A-28V_13L-7W
- added U$1, U$2: NET_BRIDGE, MrSwirlyEyes:NET_BRIDGE
- added VREG1, VREG2: 1.5A/3.3V, MrSwirlyEyes:VREGTL1963A-33DCYR_LDO_1.5A-3.3V
- added VREG3: 1.5A/2.5V, MrSwirlyEyes:VREGTL1963A-25DCYR_LDO_1.5A-2.5V
Connections:
- new net 3.3V: C65.1, C70.1, D7.A, D8.A, VREG2.VO, VREG3.VO
- new net N$38: L2.2, U$2.P$1
- new net N$40: C64.1, C66.1, C67.A, C68.1, C69.1, C71.1, C78.A, D6.K, D7.K, D8.K, SW1.S1, VREG1.VI, VREG2.VI, VREG3.VI
- new net N$43: BATT1.P, SW1.P
- new net NGND: C79.2, U$1.P$1, U$2.P$2
- net GND: now also BATT1.N, C63.2, C64.2, C65.2, C66.2, C67.K, C68.2, C69.2, C70.2, C71.2, C74.2, C78.K, L2.1, U$1.P$2, VREG1.GND, VREG2.GND, VREG3.GND
- net VCC: now also C63.1, C74.1, C79.1, D6.A, L1.1, L1.2, VREG1.VO
Other:
- note added: "LPF"
- note added: "MCU"
- note added: "Might need a second one?"
- note added: "THERMOELECTRICS"
- note added: "VIBROTACTILE DRIVERS"
- note added: "VIBROTACTILES"
- note removed: "VIBE MOTOR DRIVERS"
- moved on the sheet: C62, J1, JP1, R16, R20, R24, R28, R32

Commit message: Unity to RED board test added.  Unity to Arduino test moved.  Several changes to Touch Glove sch and brd
Parts:
- removed C76: 0.1uF/50V, MrSwirlyEyes:CAP_CERAMIC_SMD-805_0.1UF-50V-10%
- removed D8: 1A/50V, MrSwirlyEyes:DIODE_GEN-PURPSMD_GP_1A-50V-SOD123F
- removed VREG1: 1.5A/3.3V, MrSwirlyEyes:VREGTL1963A-33DCYR_LDO_1.5A-3.3V
- added C72, C77: 10uF/25V, MrSwirlyEyes:CAP_CERAMIC_SMD-805_10UF-25V-10%
- added C73, C80: 0.1uF/50V, MrSwirlyEyes:CAP_CERAMIC_SMD-805_0.1UF-50V-10%
- added C81: 100UF/16V, MrSwirlyEyes:CAP_POLARIZED_ALUM-ELECTROLYTIC_SMD_100UF-16V-20%
- added C82: 220uF/16V, MrSwirlyEyes:CAP_POLARIZED_ALUM-ELECTROLYTIC_SMD_220UF-16V-20%
- added D9: 1A/50V, MrSwirlyEyes:DIODE_GEN-PURPSMD_GP_1A-50V-SOD123F
- added VREG4: 3A/2.5V, MrSwirlyEyes:VREG_LT1764EQ_ULDO_FAST-TRANSIENTLT1764EQ-2.5_3A-2.5V
- C64, C66, C70: value 10uF/25V -> 0.1uF/50V; device MrSwirlyEyes:CAP_CERAMIC_SMD-805_10UF-25V-10% -> MrSwirlyEyes:CAP_CERAMIC_SMD-805_0.1UF-50V-10%
- C74: value 0.1uF/50V -> 10uF/25V; device MrSwirlyEyes:CAP_CERAMIC_SMD-805_0.1UF-50V-10% -> MrSwirlyEyes:CAP_CERAMIC_SMD-805_10UF-25V-10%
- VREG3: value 1.5A/2.5V -> 1A/3.3V; device MrSwirlyEyes:VREGTL1963A-25DCYR_LDO_1.5A-2.5V -> MrSwirlyEyes:VREG_TPS76833_ULDO_FAST-TRANSIENT_1A-3.3VTPS76833QDR_1A-3.3V
Connections:
- net 3.3V: now also C75.1, C77.1, C80.1, C81.A, C82.A, D9.A, VREG4.SENSE, VREG4.VOUT; no longer C70.1, D8.A, VREG3.VO
- net GND: now also C72.2, C73.2, C75.2, C77.2, C80.2, C81.K, C82.K, VREG3.!EN, VREG4.GND; no longer VREG1.GND
- net N$40: now also C72.1, C73.1, C74.1, D9.K, VREG3.VIN, VREG4.!SHDN, VREG4.VIN; no longer D8.K, VREG1.VI, VREG3.VI
- net VCC: now also C70.1, VREG3.VOUT; no longer C74.1, VREG1.VO
Other:
- note removed: "Might need a second one?"
- moved on the sheet: C62, C63, C64, C65, C66, C70, C71, C74, C75, C79, D6, D7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

Commit message: Rev 1 of Touch Glove schematic complete.  Putting Touch Glove PCB on hold until Robotic Arm schematic + PCB are done
Other:
- note removed: "NOTE: drive at 3V"
- moved on the sheet: A1, B1, BATT1, C1, C10, C11, C12, C13, C14, C15, C16, C17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

Commit message: Replaced 2.5V regulator for TECs to 1.8V regulator for TECs.  2.5V got way too hot.  But 1.8V can be used effectively
Parts:
- J1: value (none) -> AVR ISP
- VREG4: value 3A/2.5V -> 3A/1.8V; device MrSwirlyEyes:VREG_LT1764EQ_ULDO_FAST-TRANSIENTLT1764EQ-2.5_3A-2.5V -> MrSwirlyEyes:VREG_LT1764EQ_ULDO_FAST-TRANSIENTLT1764EQ-1.8_3A-1.8V
Other:
- moved on the sheet: FLEX1, FLEX2, FLEX3, FLEX4, FLEX5

Commit message: Modified code to work with new PCB board.  Removed libraries, placed in new repo.  Finished and printed Robotic Arm PCB board.  Tested and WORKS!  Started on Touch Glove PCB
Parts:
- removed A1: ANTENNASMD5, lib_kenmei:ANTENNASMD5
- removed B1: 748421245, lib_kenmei:BALUN0805
- removed C36, C38, C40, C41, C47: 1uF/25V, MrSwirlyEyes:CAP_CERAMIC_SMD-805-1UF-25V-10%
- removed C37, C39, C46, C51, C62: 0.1uF/50V, MrSwirlyEyes:CAP_CERAMIC_SMD-805_0.1UF-50V-10%
- removed C42, C43: 12pF/250V, MrSwirlyEyes:CAP_CERAMIC_SMD-805_12PF-250V-5%
- removed C44: 22PF/250V, MrSwirlyEyes:CAP_CERAMIC_SMD-805_22PF-250V-5%
- removed C45: 0.75PF/100V, MrSwirlyEyes:CAP_CERAMIC_SMD-805-0.75PF-100V-33%
- removed C48: 0.22uF/50V, MrSwirlyEyes:CAP_CERAMIC_SMD-805_0.22UF-50V-10%
- removed C49, C50: 10uF/25V, MrSwirlyEyes:CAP_CERAMIC_SMD-805_10UF-25V-10%
- removed DEMUX: CH16_MUX-DEMUX, MrSwirlyEyes:CD74HC4067-SM96_16:1_MUX-DEMUX
- removed IMU1: LM9DS1, lib_kenmei:LSM9DS1_IMU
- removed J1: AVR ISP, MrSwirlyEyes:AVR_SPI_PRG_6NS
- removed JP1: FTDIPTH-RA, MrSwirlyEyes:FTDIPTH-RA
- removed R38: 10KΩ, MrSwirlyEyes:RESISTORSMD-0805_1/8W_10K_5%
- removed U6: ATMEGA128RFA1, MrSwirlyEyes:ATMEGA128RFA1
- removed Y1: 16MHz, MrSwirlyEyes:CRYSTAL_ABM3B_16MHZ_18PF
- added A6: 2.4GHz/802.11/0.5dBi/3W, PiB_radio_frequency:ANTENNA_SMD-CHIP_2.4GHZ-0.5DBI-3W
- added ANALOG_BR, NOISE_BR: 2PT_GND_TIE, PiB_power_symbols:2PT_GND_TIE
- added AVR_ISP: AVR ISP, PiB_connectors:AVR_SPI_PRG_6NS
- added B2: Impedence UNBAL/BAL (50Ω/100Ω), PiB_radio_frequency:BALUN_SMD-0805_UNBAL/BAL-50/100
- added BATT2: BATTERYPTH_HOLES, PiB:BATTERYPTH_HOLES
- added C100, C106, C108, C116, C117, C119, C121, C122, C124, C127, C129, C135, C98: 0.1uF/50V, PiB_capacitors:0.1UF_SMD-805_50V-10%
- added C107, C109, C110, C111, C132, C134, C136: 1uF/25V, PiB_capacitors:1UF_SMD-805_25V-10%
- added C112, C113: 12pF/250V, PiB_capacitors:12PF_SMD-805_250V-5%
- added C114: 22PF/250V, PiB_capacitors:22PF_SMD-805_250V-5%
- added C115: 0.75PF/100V, PiB_capacitors:0.75PF_SMD-805_100V-33%
- added C118: 220uF/16V, PiB_capacitors:220UF-POLARIZED_SMD_16V-20%
- added C120, C123, C125, C126, C128, C97, C99: 10uF/25V, PiB_capacitors:10UF_CER_SMD-805_25V-10%
- added C133: 100UF/16V, PiB_capacitors:100UF-POLARIZED_SMD_16V-20%
- added D10, D11, D8: 1A/50V, PiB_discrete_semiconductors:DIODE_GENERAL-PURPOSE_SMD_GP_1A-50V
- added D12: 1A/50V, MrSwirlyEyes:DIODE_GEN-PURPSMD_GP_1A-50V-SOD123F
- added DEMUX1: CH16_MUX-DEMUX, PiB:CD74HC4067-SM96_16:1_MUX-DEMUX
- added J2: (ID,OD)=(2.1,5.5)MM, PiB_connectors:POWER_JACK-BARREL_ID2.1MM-OD5.5MM
- added JP2: FTDIPTH-RA, PiB_connectors:FTDIPTH-RA
- added L3, L4: 10uH, PiB_inductors:10UH_SMD-805_0.5A-0.65OHM-10%
- added L5: BLUE, PiB_leds:LED_SMD-0805_DISCRETE_BLUE
- added L6: GREEN, PiB_leds:LED_SMD-0805_DISCRETE_GREEN
- added L7: RED, PiB_leds:LED_SMD-0805_DISCRETE_RED
- added MCU: ATMEGA128RFA1, PiB_ic_microcontrollers:ATMEGA128RFA1_VFQFN-64_EXPOSED-PAD
- added PWM_DRIVER1: PCA9685, PiB:PCA9685_16-CH_12-BIT_PWM-DRIVER
- added R40, R41: 4.7K, PiB_resistors:4.7KΩ_SMD-0805_1/8W-5%
- added R46, R47: 10KΩ, PiB_resistors:10KΩ_SMD-0805_1/8W-5%
- added R48: 2KΩ, PiB_resistors:2KΩ_SMD-0805_1/8W-5%
- added R49: 1KΩ, PiB_resistors:1KΩ_SMD-0805_1/8W-5%
- added S7: TACTILE-SW_500mA/12V, PiB_switches:SWITCH_MOMENTARYSPST-SMD-50MA-12V_L5.2-W5.2
- added SW2: 5A/28V, PiB_switches:SWITCH_SPDT_VERT_PTH_5A-28V_13L-7W
- added VIBE_6: VIBE_MOTOR, MrSwirlyEyes:VIBE_MOTOR_100MA/3V
- added VIBE_T6: 2.6A/20V/57mΩ, MrSwirlyEyes:MOSFET-N-CH_SI2302CDS_2.6A_20V_57MΩ_SOT23-3
- added VREG1: 1A/3.3V, PiB_ic_power:VREG_TPS76833_ULDO_FAST-TRANSIENT_1A-3.3VTPS76833QDR_1A-3.3V
- added VREG5: 5A/5V, PiB_ic_power:VREG_MIC29501-5.0_LINEAR_ULDO_5A-5VMIC29501-5.0_5A-5V
- added Y2: 16MHz, PiB:CRYSTAL_ABM3B_16MHZ_18PF
- C1: value 10uF/25V -> 0.1uF/50V; device MrSwirlyEyes:CAP_CERAMIC_SMD-805_10UF-25V-10% -> MrSwirlyEyes:CAP_CERAMIC_SMD-805_0.1UF-50V-10%
- C35: value 0.1uF/50V -> 10uF/25V; device MrSwirlyEyes:CAP_CERAMIC_SMD-805_0.1UF-50V-10% -> MrSwirlyEyes:CAP_CERAMIC_SMD-805_10UF-25V-10%
- R12: value 4.7K -> 10KΩ; device MrSwirlyEyes:RESISTORSMD-0805_1/8W_4.7K_5% -> MrSwirlyEyes:RESISTORSMD-0805_1/8W_10K_5%
- R13: value 4.7K -> 100Ω; device MrSwirlyEyes:RESISTORSMD-0805_1/8W_4.7K_5% -> MrSwirlyEyes:RESISTORSMD-0805_1/8W_100_5%
Connections:
- removed net C5: DEMUX.C5
- removed net C6: DEMUX.C6
- removed net C7: DEMUX.C7
- removed net C8: DEMUX.C8
- removed net C9: DEMUX.C9
- removed net N$33: B1.OUT1, U6.RFP
- removed net N$34: B1.GND@2, C44.1
- removed net N$35: C42.1, U6.XTAL2, Y1.1
- removed net N$36: C49.1, IMU1.CAP
- removed net N$37: C48.1, IMU1.C1
- removed net N$39: A1.SIGNAL, B1.IN, C45.1
- removed net N$41: C62.1, JP1.2
- removed net N$42: JP1.5
- removed net S0: DEMUX.S0
- removed net S1: DEMUX.S1
- removed net S2: DEMUX.S2
- removed net S3: DEMUX.S3
- removed net SIG: DEMUX.SIG
- new net 5V: C121.1, C125.1, C133.A, D10.A, VREG5.VOUT
- new net AGND: ANALOG_BR.P$2, C100.2, C122.2, C134.2, C135.2, C136.2, C97.2, DEMUX1.!EN, DEMUX1.GND, MCU.AVSS
- new net AVCC: C100.1, C122.1, C134.1, C135.1, C136.1, C97.1, DEMUX1.VCC, L3.2, MCU.AREF, MCU.EVDD
- new net BATT_+: BATT2.P, J2.PWR, SW2.2
- new net BATT_-: BATT2.N, J2.GND@1
- new net N$44: C113.1, MCU.XTAL1, Y2.2
- new net N$45: B2.OUT2, MCU.RFN
- new net N$46: B2.OUT1, MCU.RFP
- new net N$47: B2.GND@2, C114.1
- new net N$48: C112.1, MCU.XTAL2, Y2.1
- new net N$49: A6.SIGNAL, B2.IN, C115.1
- new net N$50: C117.1, JP2.2
- new net N$51: JP2.5
- new net N$52: ANALOG_BR.P$1, L4.2
- new net N$53: L5.K, R47.2
- new net N$54: L6.K, R49.2
- new net N$55: L7.K, R48.2
- new net N$62: C132.1, MCU.DVDD
- new net N$63: C110.1, MCU.AVDD
- new net STRAIN_10: DEMUX1.C9
- new net STRAIN_6: DEMUX1.C5
- new net STRAIN_7: DEMUX1.C6
- new net STRAIN_8: DEMUX1.C7
- new net STRAIN_9: DEMUX1.C8
- new net VBATT: C118.A, C119.1, C120.1, C126.1, C127.1, C128.1, C129.1, D10.K, D8.K, L5.A, SW2.1, VREG1.VIN, VREG5.EN, VREG5.VIN
- new net VIBE_6: PWM_DRIVER.PWM15, R12.2, R13.1
- net A0: now also MCU.(ADC0/A0*)PF0; no longer U6.PF0(ADC0)
- net A1: now also MCU.(ADC1/A1*)PF1; no longer U6.PF1(ADC1)
- net A2: now also MCU.(ADC2/DIG2/A2*)PF2; no longer U6.PF2(ADC2/DIG2)
- net A3: now also MCU.(ADC3/DIG4/A3*)PF3; no longer U6.PF3(ADC3/DIG4)
- net A4: now also MCU.(ADC4/TCK/A4*)PF4; no longer U6.PF4(ADC4/TCK)
- net A5: now also DEMUX1.SIG, MCU.(ADC5/TMS/A5*)PF5; no longer U6.PF5(ADC5/TMS)
- net A6: now also MCU.(ADC6/TDO/A6*)PF6; no longer U6.PF6(ADC6/TDO)
- net A7: now also MCU.(ADC7/TDI/A7*)PF7; no longer U6.PF7(ADC7/TDI)
- net C10: now also DEMUX1.C10; no longer DEMUX.C10
- net C11: now also DEMUX1.C11; no longer DEMUX.C11
- net C12: now also DEMUX1.C12; no longer DEMUX.C12
- net C13: now also DEMUX1.C13; no longer DEMUX.C13
- net C14: now also DEMUX1.C14; no longer DEMUX.C14
- net C15: now also DEMUX1.C15; no longer DEMUX.C15
- net GND: now also AVR_ISP.6, B2.GND@5, C106.2, C107.2, C108.2, C109.2, C110.2, C111.2, C112.2, C113.2, C114.2, C115.2, C116.2, C118.K, C119.2, C120.2, C123.2, C124.2, C126.2, C127.2, C132.2, C98.2, C99.2, J2.GND@2, JP2.6, L4.1, MCU.AVSS_RFN, MCU.AVSS_RFP, MCU.CLKI, MCU.DVSS, MCU.TST, NOISE_BR.P$2, PWM_DRIVER1.!OE, PWM_DRIVER1.A0, PWM_DRIVER1.A1, PWM_DRIVER1.A2, PWM_DRIVER1.A3, PWM_DRIVER1.A4, PWM_DRIVER1.A5, PWM_DRIVER1.EXTCLK, PWM_DRIVER1.GND, R12.1, R47.1, R48.1, R49.1, S7.1, VIBE_T6.S, VREG1.!EN, VREG1.GND; no longer B1.GND@5, C1.2, C36.2, C37.2, C38.2, C39.2, C40.2, C41.2, C42.2, C43.2, C44.2, C45.2, C46.2, C47.2, C48.2, C49.2, C50.2, C51.2, DEMUX.!EN, DEMUX.GND, IMU1.GND@1, IMU1.GND@2, IMU1.RES@1, IMU1.RES@2, IMU1.RES@3, IMU1.RES@4, IMU1.RES@5, J1.6, JP1.6, U6.AVSS, U6.AVSS_RFN, U6.AVSS_RFP, U6.CLKI, U6.DVSS, U6.TST
- net MISO: now also AVR_ISP.1, MCU.(PDO/PCINT3/MISO/D12)PB3; no longer J1.1, U6.PB3(MISO/PDO/PCINT3)
- net MOSI: now also AVR_ISP.4, MCU.(PDI/PCINT2/MOSI/D11)PB2; no longer J1.4, U6.PB2(MOSI/PDI/PCINT2)
- net N$30: now also C1.2, D12.A, VIBE_6.-, VIBE_T6.D; no longer C43.1, U6.XTAL1, Y1.2
- net N$32: now also R13.2, VIBE_T6.G; no longer B1.OUT2, U6.RFN
- net NGND: now also C121.2, C125.2, C128.2, C129.2, C133.K, NOISE_BR.P$1, VREG5.GND
- net PB4: now also MCU.(PCINT4/OC2A/D9-PWM9)PB4; no longer U6.PB4(OC2A/PCINT4)
- net PB5: now also MCU.(PCINT5/OC1A/D8-PWM8)PB5; no longer U6.PB5(OC1A/PCINT5)
- net PB6: now also L7.A, MCU.(PCINT6/OC1B/D34-PWM34)PB6; no longer U6.PB6(OC1B/PCINT6)
- net PB7: now also L6.A, MCU.(PCINT7/OC0A/OC1C/D35-PWM35)PB7; no longer U6.PB7(OC0A/OC1C/PCINT7)
- net PD4: now also MCU.(ICP1/D22)PD4; no longer U6.PD4(ICP1)
- net PD5: now also MCU.(XCK1/D23)PD5; no longer U6.PD5(XCK1)
- net PD6: now also MCU.(T1/D24)PD6; no longer U6.PD6(T1)
- net PD7: now also MCU.(T0/D25)PD7; no longer U6.PD7(T0)
- net PE2: now also DEMUX1.S0, MCU.(XCK0/AIN0/D2)PE2; no longer U6.PE2(XCK0/AIN0)
- net PE3: now also MCU.(AIN1/OC3A/D3-PWM3)PE3; no longer U6.PE3(OC3A/AIN1)
- net PE4: now also MCU.(INT4/OC3B/D4-PWM4)PE4; no longer U6.PE4(OC3B/INT4)
- net PE5: now also MCU.(INT5/OC3C/D5-PWM5)PE5; no longer U6.PE5(OC3C/INT5)
- net PE6: now also DEMUX1.S1, MCU.(T3/INT6/D6)PE6; no longer U6.PE6(T3/INT6)
- net PE7: now also DEMUX1.S2, MCU.(ICP3/INT7/CLKO/D7)PE7; no longer U6.PE7(ICP3/INT7/CLKO)
- net PG0: now also MCU.(DIG3/D16)PG0; no longer U6.PG0(DIG3)
- net PG1: now also MCU.(DIG1/D17)PG1; no longer U6.PG1(DIG1)
- net PG2: now also MCU.(AMR/D18)PG2; no longer U6.PG2(AMR)
- net PG3: now also MCU.(TOSC2)PG3; no longer U6.PG3(TOSC2)
- net PG4: now also MCU.(TOSC1)PG4; no longer U6.PG4(TOSC1)
- net PG5: now also MCU.(OC0B/D19-PWM19)PG5; no longer U6.PG5(OC0B)
- net PWM10: now also PWM_DRIVER1.PWM10; no longer PWM_DRIVER.PWM10
- net RESET: now also AVR_ISP.5, C117.2, D11.A, MCU.RSTN, R46.1, S7.2; no longer C62.2, J1.5, R38.1, U6.RSTN
- net RX0: now also JP2.4, MCU.(PCINT8/RXD0/D0)PE0; no longer JP1.4, U6.PE0(RXD0/PCINT8)
- net RX1: now also MCU.(INT2/RXD1/D20)PD2; no longer U6.PD2(RXD1/INT2)
- net SCK: now also AVR_ISP.3, MCU.(PCINT1/SCK/D13)PB1; no longer J1.3, U6.PB1(SCK/PCINT1)
- net SCL: now also MCU.(INT0/SCL/D15)PD0, PWM_DRIVER1.SCL, R40.1; no longer IMU1.SCL/SPC, R12.1, U6.PD0(SCL/INT0)
- net SDA: now also MCU.(INT1/SDA/D14)PD1, PWM_DRIVER1.SDA, R41.1; no longer IMU1.SDA/SDI/SDO, R13.1, U6.PD1(SDA/INT1)
- net SSN: now also DEMUX1.S3, MCU.(PCINT0/SSN/D10)PB0; no longer U6.PB0(SSN/PCINT0)
- net STRAIN_1: now also DEMUX1.C0; no longer DEMUX.C0
- net STRAIN_2: now also DEMUX1.C1; no longer DEMUX.C1
- net STRAIN_3: now also DEMUX1.C2; no longer DEMUX.C2
- net STRAIN_4: now also DEMUX1.C3; no longer DEMUX.C3
- net STRAIN_5: now also DEMUX1.C4; no longer DEMUX.C4
- net TEC_1_COLD: now also PWM_DRIVER1.PWM1
- net TEC_1_HOT: now also PWM_DRIVER1.PWM0
- net TEC_2_COLD: now also PWM_DRIVER1.PWM3
- net TEC_2_HOT: now also PWM_DRIVER1.PWM2
- net TEC_3_COLD: now also PWM_DRIVER1.PWM5
- net TEC_3_HOT: now also PWM_DRIVER1.PWM4
- net TEC_4_COLD: now also PWM_DRIVER1.PWM7
- net TEC_4_HOT: now also PWM_DRIVER1.PWM6
- net TEC_5_COLD: now also PWM_DRIVER1.PWM9
- net TEC_5_HOT: now also PWM_DRIVER1.PWM8
- net TX0: now also JP2.3, MCU.(TXD0/D1)PE1; no longer JP1.3, U6.PE1(TXD0)
- net TX1: now also MCU.(INT3/TXD1/D21)PD3; no longer U6.PD3(TXD1/INT3)
- net VCC: now also AVR_ISP.2, C106.1, C107.1, C108.1, C109.1, C111.1, C116.1, C123.1, C124.1, C98.1, C99.1, D11.K, D12.K, D8.A, JP2.1, L3.1, MCU.DEVDD, PWM_DRIVER1.VCC, R40.2, R41.2, R46.2, VIBE_6.+, VREG1.VOUT; no longer C36.1, C37.1, C38.1, C39.1, C40.1, C41.1, C46.1, C47.1, C50.1, C51.1, DEMUX.VCC, IMU1.VDD@1, IMU1.VDD@2, IMU1.VDDIO@1, IMU1.VDDIO@2, J1.2, JP1.1, R12.2, R13.2, R38.2, U6.AREF, U6.AVDD, U6.DEVDD, U6.DVDD, U6.EVDD
- net VIBE_1: now also PWM_DRIVER.PWM10, PWM_DRIVER1.PWM11; no longer PWM_DRIVER.PWM11
- net VIBE_2: now also PWM_DRIVER.PWM11, PWM_DRIVER1.PWM12; no longer PWM_DRIVER.PWM12
- net VIBE_3: now also PWM_DRIVER.PWM12, PWM_DRIVER1.PWM13; no longer PWM_DRIVER.PWM13
- net VIBE_4: now also PWM_DRIVER.PWM13, PWM_DRIVER1.PWM14; no longer PWM_DRIVER.PWM14
- net VIBE_5: now also PWM_DRIVER.PWM14, PWM_DRIVER1.PWM15; no longer PWM_DRIVER.PWM15
Other:
- note added: "A0/0 --> SIG_PIN of DEMUX"
- note added: "ANALOG DEMUX"
- note added: "CHANGE TO 470 UF"
- note added: "D10"
- note added: "D10 --> S3 of DEMUX"
- note added: "D2"
- note added: "D2 --> S0 of DEMUX"
- note added: "D6"
- note added: "D6 --> S1 of DEMUX"
- note added: "D7"
- note added: "D7 --> S2 of DEMUX"
- note added: "POWER SYSTEM"
- note added: "PWM DRIVER"
- note added: "ROBOTIC ARM"
- note added: "Rev 1"
- note added: "SERVOS"
- note added: "TODO: LOTS OF VIAS"
- note added: "TRANSMISSION OF TOUCH VR"
- note added: "add diode CD1206-S01575"
- note removed: "DEMULTIPLEXER"
- note removed: "IMU LM9DS1"
- moved on the sheet: C1, C24, C35, R12, R13

Commit message: Started on Touch Glove.  Going full ambitious using 0402 for resistors, capacitors, and inductors
Parts:
- removed BATT1: BATTERYPTH_HOLES, MrSwirlyEyes:BATTERYPTH_HOLES
- removed C121, C129: 0.1uF/50V, PiB_capacitors:0.1UF_SMD-805_50V-10%
- removed C125, C128: 10uF/25V, PiB_capacitors:10UF_CER_SMD-805_25V-10%
- removed C133: 100UF/16V, PiB_capacitors:100UF-POLARIZED_SMD_16V-20%
- removed C2, C64, C66, C68, C70, C73, C75, C80: 0.1uF/50V, MrSwirlyEyes:CAP_CERAMIC_SMD-805_0.1UF-50V-10%
- removed C23, C63, C65, C69, C71, C72, C74, C77: 10uF/25V, MrSwirlyEyes:CAP_CERAMIC_SMD-805_10UF-25V-10%
- removed C67, C82: 220uF/16V, MrSwirlyEyes:CAP_POLARIZED_ALUM-ELECTROLYTIC_SMD_220UF-16V-20%
- removed C78, C81: 100UF/16V, MrSwirlyEyes:CAP_POLARIZED_ALUM-ELECTROLYTIC_SMD_100UF-16V-20%
- removed C79: 1uF/25V, MrSwirlyEyes:CAP_CERAMIC_SMD-805-1UF-25V-10%
- removed D10: 1A/50V, PiB_discrete_semiconductors:DIODE_GENERAL-PURPOSE_SMD_GP_1A-50V
- removed D6, D7, D9: 1A/50V, MrSwirlyEyes:DIODE_GEN-PURPSMD_GP_1A-50V-SOD123F
- removed J2: (ID,OD)=(2.1,5.5)MM, PiB_connectors:POWER_JACK-BARREL_ID2.1MM-OD5.5MM
- removed L1, L2: 10uH, MrSwirlyEyes:INDUCTORSMD-805_10UH-0.5A-0.65OHM-10%
- removed P1, P2, P3, P4, P5: PELTIER, MrSwirlyEyes:PELTIER-TECNL1025T_1.8A-4.4V_L10.7-W8.8-H2
- removed PWM_DRIVER: PCA9685, MrSwirlyEyes:PCA9685_16-CH_12-BIT_PWM-DRIVER
- removed SW1: 5A/28V, MrSwirlyEyes:SWITCH_SPDT5A-28V_13L-7W
- removed U$1, U$2: NET_BRIDGE, MrSwirlyEyes:NET_BRIDGE
- removed U1, U2, U3, U4, U5: DRV8837C, MrSwirlyEyes:DRV8837C_H-BRIDGE_1A_WSON-8-PADDRV8837C_1A
- removed VIBE_1, VIBE_2, VIBE_3, VIBE_4, VIBE_5, VIBE_6: VIBE_MOTOR, MrSwirlyEyes:VIBE_MOTOR_100MA/3V
- removed VIBE_T1, VIBE_T2, VIBE_T3, VIBE_T4, VIBE_T5, VIBE_T6: 2.6A/20V/57mΩ, MrSwirlyEyes:MOSFET-N-CH_SI2302CDS_2.6A_20V_57MΩ_SOT23-3
- removed VREG2: 1.5A/3.3V, MrSwirlyEyes:VREGTL1963A-33DCYR_LDO_1.5A-3.3V
- removed VREG3: 1A/3.3V, MrSwirlyEyes:VREG_TPS76833_ULDO_FAST-TRANSIENT_1A-3.3VTPS76833QDR_1A-3.3V
- removed VREG4: 3A/1.8V, MrSwirlyEyes:VREG_LT1764EQ_ULDO_FAST-TRANSIENTLT1764EQ-1.8_3A-1.8V
- removed VREG5: 5A/5V, PiB_ic_power:VREG_MIC29501-5.0_LINEAR_ULDO_5A-5VMIC29501-5.0_5A-5V
- added C36, C38, C40, C45, C47, C48, C49, C50, C51: 0.1uF/50V, PiB_capacitors:0.1UF_SMD-0402_50V-10%
- added C37, C44: 10uF/16V, PiB_capacitors:10UF_CER_SMD-603_16V-10%
- added C39, C43: 10uF/10V, PiB_capacitors:10UF_CER_SMD-0402_10V-20%
- added C41, C42, C46: 100uF, PiB_capacitors:100UF_CER_SMD-1210_16V-20%
- added D13, D14: 1A/50V, MrSwirlyEyes:DIODE_GEN-PURPSMD_GP_1A-50V-SOD123F
- added FLEX10, FLEX6, FLEX7, FLEX8, FLEX9: 10K, PiB:FLEX-SENSOR10K_2.2IN
- added HBRIDGE1, HBRIDGE2, HBRIDGE3, HBRIDGE4, HBRIDGE5: DRV8837C, PiB:DRV883X_H-BRIDGE_DRV8837C_1A
- added Q1, Q2, Q3, Q4, Q5, Q6: MCH3474 4A/30V/50mΩ, PiB_discrete_semiconductors:POWER_NCHAN_MCH3474
- added R38, R39, R42, R43, R44: 10KΩ, PiB_resistors:10KΩ_SMD-0402_1/16W-5%
- added TEC1, TEC2, TEC3, TEC4, TEC5: PELTIER, PiB:PELTIER-TECNL1025T_1.8A-4.4V_L10.7-W8.8-H2
- added VIBE1, VIBE2, VIBE3, VIBE4, VIBE5, VIBE6: VIBE_MOTOR, PiB:VIBE_MOTOR_100MA/3V
- added VREG6: TL1963A-33 1.5A/3.3V, PiB_ic_power:VREG_LINEAR_FIXED_TL1963A-33_LDO_1.5A-3.3V
- added VREG7: 3A/1.8V, MrSwirlyEyes:VREG_LT1764EQ_ULDO_FAST-TRANSIENTLT1764EQ-1.8_3A-1.8V
- C1, C12, C13, C16, C17, C20, C21, C24, C25, C26, C3, C30, C31, C32, C33, C34, C4, C5, C52, C53, C54, C55, C56, C6, C7, C8, C9: device MrSwirlyEyes:CAP_CERAMIC_SMD-805_0.1UF-50V-10% -> PiB_capacitors:0.1UF_SMD-0402_50V-10%
- C10, C11, C14, C15, C18, C19, C22, C27, C28, C29, C35, C57, C58, C59, C60, C61: value 10uF/25V -> 10uF/10V; device MrSwirlyEyes:CAP_CERAMIC_SMD-805_10UF-25V-10% -> PiB_capacitors:10UF_CER_SMD-0402_10V-20%
- C100, C106, C108, C116, C117, C119, C122, C124, C127, C135, C98: device PiB_capacitors:0.1UF_SMD-805_50V-10% -> PiB_capacitors:0.1UF_SMD-0402_50V-10%
- C107, C109, C110, C111, C132, C134, C136: device PiB_capacitors:1UF_SMD-805_25V-10% -> PiB_capacitors:1UF_CER_SMD-603_25V-10%
- C118: value 220uF/16V -> 100uF; device PiB_capacitors:220UF-POLARIZED_SMD_16V-20% -> PiB_capacitors:100UF_CER_SMD-1210_16V-20%
- C120, C126: value 10uF/25V -> 10uF/16V; device PiB_capacitors:10UF_CER_SMD-805_25V-10% -> PiB_capacitors:10UF_CER_SMD-603_16V-10%
- C123, C97, C99: value 10uF/25V -> 10uF/10V; device PiB_capacitors:10UF_CER_SMD-805_25V-10% -> PiB_capacitors:10UF_CER_SMD-0402_10V-20%
- D1, D12, D2, D3, D4, D5: value 1A/50V -> 150mA/75V; device MrSwirlyEyes:DIODE_GEN-PURPSMD_GP_1A-50V-SOD123F -> PiB_discrete_semiconductors:DIODE_GENERAL-PURPOSE_SMD-0402_GP_120MA-75V
- FLEX1, FLEX2, FLEX3, FLEX4, FLEX5: device MrSwirlyEyes:FLEX-SENSOR10K_2.2IN -> PiB:FLEX-SENSOR10K_2.2IN
- L5: device PiB_leds:LED_SMD-0805_DISCRETE_BLUE -> PiB_leds:LED_SMD-0603_DISCRETE_BLUE
- R1, R11, R12, R14, R16, R18, R2, R20, R22, R24, R26, R28, R3, R30, R32, R34, R35, R36, R37, R4, R5: device MrSwirlyEyes:RESISTORSMD-0805_1/8W_10K_5% -> PiB_resistors:10KΩ_SMD-0402_1/16W-5%
- R10, R13, R15, R17, R19, R21, R23, R25, R27, R29, R31, R33, R6, R7, R8, R9: device MrSwirlyEyes:RESISTORSMD-0805_1/8W_100_5% -> PiB_resistors:100Ω_SMD-0402_1/16W-5%
- R46, R47: device PiB_resistors:10KΩ_SMD-0805_1/8W-5% -> PiB_resistors:10KΩ_SMD-0402_1/16W-5%
Connections:
- removed net 5V: C121.1, C125.1, C133.A, D10.A, VREG5.VOUT
- removed net BATT_-: BATT2.N, J2.GND@1
- removed net C14: DEMUX1.C14
- removed net C15: DEMUX1.C15
- removed net FSR_1: FLEX1.-, R11.2
- removed net FSR_2: FLEX2.-, R34.2
- removed net FSR_3: FLEX3.-, R35.2
- removed net FSR_4: FLEX4.-, R36.2
- removed net FSR_5: FLEX5.-, R37.2
- removed net N$38: L2.2, U$2.P$1
- removed net N$40: C64.1, C66.1, C67.A, C68.1, C69.1, C71.1, C72.1, C73.1, C74.1, C78.A, D6.K, D7.K, D9.K, SW1.S1, VREG2.VI, VREG3.VIN, VREG4.!SHDN, VREG4.VIN
- removed net N$43: BATT1.P, SW1.P
- removed net PWM10: PWM_DRIVER1.PWM10
- removed net VM: C10.1, C13.1, C14.1, C17.1, C18.1, C21.1, C22.1, C26.1, C27.1, C9.1, U1.VM, U2.VM, U3.VM, U4.VM, U5.VM
- new net 1.8V: C10.1, C13.1, C14.1, C17.1, C18.1, C21.1, C22.1, C26.1, C27.1, C39.1, C40.1, C42.1, C9.1, D14.A, HBRIDGE1.VM, HBRIDGE2.VM, HBRIDGE3.VM, HBRIDGE4.VM, HBRIDGE5.VM, VREG7.SENSE, VREG7.VOUT
- new net C8: DEMUX1.C8
- new net C9: DEMUX1.C9
- net 3.3V: now also C1.1, C24.1, C3.1, C35.1, C36.1, C4.1, C41.1, C43.1, C5.1, C52.1, C53.1, C54.1, C55.1, C56.1, C57.1, C58.1, C59.1, C6.1, C60.1, C61.1, C7.1, D1.K, D12.K, D13.A, D2.K, D3.K, D4.K, D5.K, VIBE1.+, VIBE2.+, VIBE3.+, VIBE4.+, VIBE5.+, VIBE6.+, VREG6.VO; no longer C65.1, C75.1, C77.1, C80.1, C81.A, C82.A, D7.A, D9.A, VREG2.VO, VREG4.SENSE, VREG4.VOUT
- net AGND: now also C30.2, C31.2, C32.2, C33.2, C34.2, C47.2, C48.2, C49.2, C50.2, C51.2, R11.1, R34.1, R35.1, R36.1, R37.1, R38.1, R39.1, R42.1, R43.1, R44.1
- net AVCC: now also C30.1, C31.1, C32.1, C33.1, C34.1, C47.1, C48.1, C49.1, C50.1, C51.1, FLEX1.+, FLEX10.+, FLEX2.+, FLEX3.+, FLEX4.+, FLEX5.+, FLEX6.+, FLEX7.+, FLEX8.+, FLEX9.+
- net BATT_+: no longer J2.PWR
- net GND: now also BATT2.N, C118.2, C36.2, C37.2, C38.2, C39.2, C40.2, C41.2, C42.2, C43.2, C44.2, C45.2, C46.2, VREG6.GND, VREG7.GND; no longer BATT1.N, C10.2, C118.K, C13.2, C14.2, C17.2, C18.2, C2.2, C21.2, C22.2, C23.2, C24.2, C26.2, C27.2, C30.2, C31.2, C32.2, C33.2, C34.2, C35.2, C52.2, C53.2, C54.2, C55.2, C56.2, C57.2, C58.2, C59.2, C60.2, C61.2, C63.2, C64.2, C65.2, C66.2, C67.K, C68.2, C69.2, C70.2, C71.2, C72.2, C73.2, C74.2, C75.2, C77.2, C78.K, C80.2, C81.K, C82.K, C9.2, J2.GND@2, L2.1, PWM_DRIVER.!OE, PWM_DRIVER.A0, PWM_DRIVER.A1, PWM_DRIVER.A2, PWM_DRIVER.A3, PWM_DRIVER.A4, PWM_DRIVER.A5, PWM_DRIVER.EXTCLK, PWM_DRIVER.GND, R1.1, R11.1, R12.1, R2.1, R3.1, R34.1, R35.1, R36.1, R37.1, R4.1, R5.1, U$1.P$2, U1.GND, U2.GND, U3.GND, U4.GND, U5.GND, VIBE_T1.S, VIBE_T2.S, VIBE_T3.S, VIBE_T4.S, VIBE_T5.S, VIBE_T6.S, VREG2.GND, VREG3.!EN, VREG3.GND, VREG4.GND
- net N$1: now also HBRIDGE5.OUT2, TEC5.HOT; no longer P1.HOT, U1.OUT1
- net N$10: now also HBRIDGE4.IN1, R16.2; no longer U1.IN1
- net N$11: now also HBRIDGE4.OUT2, TEC4.HOT; no longer P2.HOT, U2.OUT1
- net N$12: now also HBRIDGE3.OUT2, TEC3.HOT; no longer P2.COLD, U2.OUT2
- net N$13: now also HBRIDGE3.IN2, R18.2; no longer U2.IN2
- net N$14: now also HBRIDGE3.IN1, R20.2; no longer U2.IN1
- net N$15: now also Q2.D, VIBE2.-; no longer VIBE_2.-, VIBE_T2.D
- net N$16: now also HBRIDGE3.OUT1, TEC3.COLD; no longer P3.HOT, U3.OUT1
- net N$17: now also Q1.D, VIBE1.-; no longer VIBE_1.-, VIBE_T1.D
- net N$18: now also HBRIDGE2.OUT2, TEC2.HOT; no longer P3.COLD, U3.OUT2
- net N$19: now also HBRIDGE2.IN2, R22.2; no longer U3.IN2
- net N$2: now also Q4.D, VIBE4.-; no longer VIBE_4.-, VIBE_T4.D
- net N$20: now also HBRIDGE2.IN1, R24.2; no longer U3.IN1
- net N$21: now also Q4.G, R4.2; no longer VIBE_T4.G
- net N$22: now also Q5.G, R5.2; no longer VIBE_T5.G
- net N$23: now also HBRIDGE2.OUT1, TEC2.COLD; no longer P5.HOT, U5.OUT1
- net N$24: now also HBRIDGE1.OUT2, TEC1.HOT; no longer P5.COLD, U5.OUT2
- net N$25: now also HBRIDGE1.IN2, R26.2; no longer U5.IN2
- net N$26: now also HBRIDGE1.IN1, R28.2; no longer U5.IN1
- net N$27: now also HBRIDGE1.OUT1, TEC1.COLD; no longer P4.HOT, U4.OUT1
- net N$28: now also Q1.G, R1.2, R6.2; no longer P4.COLD, U4.OUT2
- net N$29: now also HBRIDGE5.IN2, R30.2; no longer U4.IN2
- net N$3: now also Q5.D, VIBE5.-; no longer VIBE_5.-, VIBE_T5.D
- net N$30: now also Q6.D, VIBE6.-; no longer VIBE_6.-, VIBE_T6.D
- net N$31: now also HBRIDGE5.IN1, R32.2; no longer U4.IN1
- net N$32: now also Q6.G, R12.2; no longer VIBE_T6.G
- net N$4: now also Q3.D, VIBE3.-; no longer VIBE_3.-, VIBE_T3.D
- net N$5: now also HBRIDGE5.OUT1, TEC5.COLD; no longer P1.COLD, U1.OUT2
- net N$6: now also HBRIDGE4.OUT1, TEC4.COLD; no longer R6.2, VIBE_T1.G
- net N$7: now also Q2.G, R2.2; no longer VIBE_T2.G
- net N$8: now also HBRIDGE4.IN2, R14.2; no longer U1.IN2
- net N$9: now also Q3.G, R3.2; no longer VIBE_T3.G
- net NGND: now also C10.2, C13.2, C14.2, C17.2, C18.2, C21.2, C22.2, C24.2, C26.2, C27.2, C35.2, C52.2, C53.2, C54.2, C55.2, C56.2, C57.2, C58.2, C59.2, C60.2, C61.2, C9.2, HBRIDGE1.GND, HBRIDGE2.GND, HBRIDGE3.GND, HBRIDGE4.GND, HBRIDGE5.GND, Q1.S, Q2.S, Q3.S, Q4.S, Q5.S, Q6.S, R1.1, R12.1, R2.1, R3.1, R4.1, R5.1; no longer C121.2, C125.2, C128.2, C129.2, C133.K, C79.2, U$1.P$1, U$2.P$2, VREG5.GND
- net SCL: no longer PWM_DRIVER.SCL
- net SDA: no longer PWM_DRIVER.SDA
- net STRAIN_1: now also FLEX3.-, R35.2
- net STRAIN_10: now also DEMUX1.C15, FLEX4.-, R36.2; no longer DEMUX1.C9
- net STRAIN_2: now also FLEX2.-, R34.2
- net STRAIN_3: now also FLEX1.-, R11.2
- net STRAIN_4: now also FLEX10.-, R44.2
- net STRAIN_5: now also FLEX9.-, R43.2
- net STRAIN_6: now also FLEX8.-, R42.2
- net STRAIN_7: now also FLEX7.-, R39.2
- net STRAIN_8: now also FLEX6.-, R38.2
- net STRAIN_9: now also DEMUX1.C14, FLEX5.-, R37.2; no longer DEMUX1.C8
- net TEC_1_COLD: now also PWM_DRIVER1.PWM11; no longer PWM_DRIVER.PWM1, PWM_DRIVER1.PWM1, R26.2
- net TEC_1_HOT: now also PWM_DRIVER1.PWM10; no longer PWM_DRIVER.PWM0, PWM_DRIVER1.PWM0, R28.2
- net TEC_2_COLD: now also PWM_DRIVER1.PWM13; no longer PWM_DRIVER.PWM3, PWM_DRIVER1.PWM3, R22.2
- net TEC_2_HOT: now also PWM_DRIVER1.PWM12; no longer PWM_DRIVER.PWM2, PWM_DRIVER1.PWM2, R24.2
- net TEC_3_COLD: now also PWM_DRIVER1.PWM15; no longer PWM_DRIVER.PWM5, PWM_DRIVER1.PWM5, R18.2
- net TEC_3_HOT: now also PWM_DRIVER1.PWM14; no longer PWM_DRIVER.PWM4, PWM_DRIVER1.PWM4, R20.2
- net TEC_4_COLD: no longer PWM_DRIVER.PWM7, R14.2
- net TEC_4_HOT: no longer PWM_DRIVER.PWM6, R16.2
- net TEC_5_COLD: no longer PWM_DRIVER.PWM9, R30.2
- net TEC_5_HOT: no longer PWM_DRIVER.PWM8, R32.2
- net VBATT: now also C118.1, C37.1, C38.1, C44.1, C45.1, C46.1, D13.K, D14.K, VREG6.VI, VREG7.!SHDN, VREG7.VIN; no longer C118.A, C128.1, C129.1, D10.K, VREG5.EN, VREG5.VIN
- net VCC: now also HBRIDGE1.NSLEEP, HBRIDGE1.VCC, HBRIDGE2.NSLEEP, HBRIDGE2.VCC, HBRIDGE3.NSLEEP, HBRIDGE3.VCC, HBRIDGE4.NSLEEP, HBRIDGE4.VCC, HBRIDGE5.NSLEEP, HBRIDGE5.VCC; no longer C1.1, C2.1, C23.1, C24.1, C3.1, C30.1, C31.1, C32.1, C33.1, C34.1, C35.1, C4.1, C5.1, C52.1, C53.1, C54.1, C55.1, C56.1, C57.1, C58.1, C59.1, C6.1, C60.1, C61.1, C63.1, C7.1, C70.1, C79.1, D1.K, D12.K, D2.K, D3.K, D4.K, D5.K, D6.A, FLEX1.+, FLEX2.+, FLEX3.+, FLEX4.+, FLEX5.+, L1.1, L1.2, PWM_DRIVER.VCC, U1.NSLEEP, U1.VCC, U2.NSLEEP, U2.VCC, U3.NSLEEP, U3.VCC, U4.NSLEEP, U4.VCC, U5.NSLEEP, U5.VCC, VIBE_1.+, VIBE_2.+, VIBE_3.+, VIBE_4.+, VIBE_5.+, VIBE_6.+, VREG3.VOUT
- net VIBE_1: now also PWM_DRIVER1.PWM0; no longer PWM_DRIVER.PWM10, PWM_DRIVER1.PWM11, R1.2
- net VIBE_2: now also PWM_DRIVER1.PWM1; no longer PWM_DRIVER.PWM11, PWM_DRIVER1.PWM12, R2.2
- net VIBE_3: now also PWM_DRIVER1.PWM2; no longer PWM_DRIVER.PWM12, PWM_DRIVER1.PWM13, R3.2
- net VIBE_4: now also PWM_DRIVER1.PWM3; no longer PWM_DRIVER.PWM13, PWM_DRIVER1.PWM14, R4.2
- net VIBE_5: now also PWM_DRIVER1.PWM4; no longer PWM_DRIVER.PWM14, PWM_DRIVER1.PWM15, R5.2
- net VIBE_6: now also PWM_DRIVER1.PWM5; no longer PWM_DRIVER.PWM15, R12.2
Other:
- note removed: "CHANGE TO 470 UF"
- note removed: "Maybe one for palm?"
- note removed: "POWER"
- note removed: "PWM DRIVER [TEC + VIBE]"
- note removed: "SERVOS"
- moved on the sheet: A6, ANALOG_BR, AVR_ISP, B2, BATT2, C1, C10, C100, C106, C107, C108, C109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

Commit message: Touch Glove Rev 1: Restarted board.  Layout for DEMUX + FLEX sensors completed
Parts:
- removed C11, C15, C19, C28, C29: 10uF/10V, PiB_capacitors:10UF_CER_SMD-0402_10V-20%
- R11, R34, R35, R36, R37, R38, R39, R42, R43, R44: value 10KΩ -> 47KΩ; device PiB_resistors:10KΩ_SMD-0402_1/16W-5% -> PiB_resistors:47KΩ_SMD-0402_1/16W-5%
Connections:
- net GND: no longer C11.2, C15.2, C19.2, C28.2, C29.2
- net STRAIN_1: now also FLEX2.-, R34.2; no longer FLEX3.-, R35.2
- net STRAIN_10: now also FLEX6.-, R38.2; no longer FLEX4.-, R36.2
- net STRAIN_2: now also FLEX7.-, R39.2; no longer FLEX2.-, R34.2
- net STRAIN_3: now also FLEX3.-, R35.2; no longer FLEX1.-, R11.2
- net STRAIN_4: now also FLEX8.-, R42.2; no longer FLEX10.-, R44.2
- net STRAIN_5: now also FLEX4.-, R36.2; no longer FLEX9.-, R43.2
- net STRAIN_6: now also FLEX9.-, R43.2; no longer FLEX8.-, R42.2
- net STRAIN_7: now also FLEX5.-, R37.2; no longer FLEX7.-, R39.2
- net STRAIN_8: now also FLEX10.-, R44.2; no longer FLEX6.-, R38.2
- net STRAIN_9: now also FLEX1.-, R11.2; no longer FLEX5.-, R37.2
- net VCC: no longer C11.1, C15.1, C19.1, C28.1, C29.1

Commit message: Touch Glove Rev 1: Routed Vibe motor, TEC + H Bridge, and PWM Driver
Parts:
- removed C24, C52, C53, C54, C55, C56: 0.1uF/50V, PiB_capacitors:0.1UF_SMD-0402_50V-10%
Connections:
- net 3.3V: no longer C24.1, C52.1, C53.1, C54.1, C55.1, C56.1
- net NGND: no longer C24.2, C52.2, C53.2, C54.2, C55.2, C56.2
- net TEC_1_COLD: now also PWM_DRIVER1.PWM6; no longer PWM_DRIVER1.PWM11
- net TEC_1_HOT: now also PWM_DRIVER1.PWM7; no longer PWM_DRIVER1.PWM10
- net TEC_2_COLD: now also PWM_DRIVER1.PWM14; no longer PWM_DRIVER1.PWM13
- net TEC_2_HOT: now also PWM_DRIVER1.PWM15; no longer PWM_DRIVER1.PWM12
- net TEC_3_COLD: now also PWM_DRIVER1.PWM12; no longer PWM_DRIVER1.PWM15
- net TEC_3_HOT: now also PWM_DRIVER1.PWM13; no longer PWM_DRIVER1.PWM14
- net TEC_4_COLD: now also PWM_DRIVER1.PWM10; no longer PWM_DRIVER1.PWM7
- net TEC_4_HOT: now also PWM_DRIVER1.PWM11; no longer PWM_DRIVER1.PWM6
- net TEC_5_COLD: now also PWM_DRIVER1.PWM8; no longer PWM_DRIVER1.PWM9
- net TEC_5_HOT: now also PWM_DRIVER1.PWM9; no longer PWM_DRIVER1.PWM8
