File: eagle/touch_glove/touch_glove.sch (EAGLE design)
At the start: 181 parts, among them Q1 MCH3474 4A/30V/50mΩ, Q2 MCH3474 4A/30V/50mΩ, Q3 MCH3474 4A/30V/50mΩ, Q4 MCH3474 4A/30V/50mΩ, Q5 MCH3474 4A/30V/50mΩ, Q6 MCH3474 4A/30V/50mΩ, SW1 4A/28V, Y2 16MHz

Commit message: Modify code to work with new PCB.  Update components on PCB due to new attributes (DISTLINK) for passive components
Parts:
- removed FLEX10: 10K, PiB:FLEX-SENSOR10K_2.2IN
- added FLEX100: 10K, PiB:FLEX-SENSOR10K_2.2IN
Connections:
- net AVCC: now also FLEX100.+; no longer FLEX10.+
- net STRAIN_1: now also FLEX1.-; no longer FLEX2.-
- net STRAIN_10: now also FLEX100.-; no longer FLEX6.-
- net STRAIN_2: now also FLEX2.-; no longer FLEX7.-
- net STRAIN_4: now also FLEX4.-; no longer FLEX8.-
- net STRAIN_5: now also FLEX5.-; no longer FLEX4.-
- net STRAIN_6: now also FLEX6.-; no longer FLEX9.-
- net STRAIN_7: now also FLEX7.-; no longer FLEX5.-
- net STRAIN_8: now also FLEX8.-; no longer FLEX10.-
- net STRAIN_9: now also FLEX9.-; no longer FLEX1.-
Other:
- moved on the sheet: FLEX1, FLEX2, FLEX4, FLEX5, FLEX6, FLEX7, FLEX8, FLEX9
