File: eagle/robotic_arm/robotic_arm.brd (EAGLE design)
At the start: 101.6 x 63.5 mm, 99 parts, among them J2 (ID,OD)=(2.1,5.5)MM, SW1 5A/28V, U6 ATMEGA128RFA1, Y1 16MHz

Commit message: Rev 1: Robotic Arm.  Initial placement of board complete at (3.30x2.50)in or (83.85x63.50)mm.  Might consider putting components on the bottom side of the board
Parts:
- removed C64: 1uF/25V, MrSwirlyEyes:CAP_CER_SMD-805
- removed FSR1, FSR2, FSR3, FSR4, FSR5: FSR, MrSwirlyEyes:CONNECTOR_FSR
- removed S1, S2, S3, S4, S5, S6: HK15298B, MrSwirlyEyes:CONNECTOR_SERVO
- removed TEMP1, TEMP2, TEMP3, TEMP4, TEMP5: TMP36, MrSwirlyEyes:CONNECTOR_TMP36
- removed U6: ATMEGA128RFA1, MrSwirlyEyes:VFQFN-64
- added FSR_INDEX, FSR_MIDDLE, FSR_PINKY, FSR_RING, FSR_THUMB: FSR, MrSwirlyEyes:CONNECTOR_FSR
- added MCU: ATMEGA128RFA1, MrSwirlyEyes:VFQFN-64
- added SERVO_INDEX, SERVO_MIDDLE, SERVO_PINKY, SERVO_RING, SERVO_THUMB, SERVO_WRIST: HK15298B, MrSwirlyEyes:CONNECTOR_SERVO
- added TEMP_INDEX, TEMP_MIDDLE, TEMP_PINKY, TEMP_RING, TEMP_THUMB: TMP36, MrSwirlyEyes:CONNECTOR_TMP36
- moved L2 356.5 mm to (73.7, 43.2), turned to 90 degrees
- moved R42 345.5 mm to (82.3, 49.8), turned to 90 degrees
- moved R41 343.9 mm to (77.0, 49.8), turned to 90 degrees
- moved R40 342.4 mm to (71.6, 49.8), turned to 90 degrees
- moved R39 340.9 mm to (66.3, 49.8), turned to 90 degrees
- moved BATT1 334.1 mm to (81.3, 42.7), turned to 270 degrees
- moved C54 327.6 mm to (29.2, 37.6), turned to 270 degrees
- moved SW1 327.2 mm to (76.7, 34.5)
- moved D1 325.8 mm to (19.3, 23.1), turned to 270 degrees
- moved C26 321.6 mm to (49.8, 43.4)
- moved C58 318.0 mm to (18.8, 32.3), turned to 270 degrees
- moved U$1 317.7 mm to (63.5, 21.6), flipped to the bottom
- moved U$2 315.5 mm to (63.5, 24.1), flipped to the bottom
- moved C63 315.1 mm to (26.4, 51.8), turned to 90 degrees
- moved C81 313.6 mm to (68.6, 36.6), turned to 90 degrees
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Connections:
- removed net 3.3V: C83.1, C94.1, D7.A, VREG1.4
- new net AGND: C18.2, C26.2, C3.2, C4.2, C47.2, C48.2, C49.2, C5.2, C50.2, C51.2, C6.2, C7.2, C85.2, DEMUX1.12, DEMUX1.15, MCU.58, MCU.61, R16.1, R39.1, R40.1, R41.1, R42.1, TEMP_INDEX.3, TEMP_MIDDLE.3, TEMP_PINKY.3, TEMP_RING.3, TEMP_THUMB.3, U$2.P$2
- new net AVCC: C18.1, C26.1, C3.1, C4.1, C47.1, C48.1, C49.1, C5.1, C50.1, C51.1, C56.1, C57.1, C6.1, C7.1, C85.1, DEMUX1.24, FSR_INDEX.+, FSR_MIDDLE.+, FSR_PINKY.+, FSR_RING.+, FSR_THUMB.+, L1.2, MCU.59, MCU.60, MCU.62, TEMP_INDEX.1, TEMP_MIDDLE.1, TEMP_PINKY.1, TEMP_RING.1, TEMP_THUMB.1
- net 5V: now also C83.1, C94.1, D7.A, SERVO_INDEX.2, SERVO_MIDDLE.2, SERVO_PINKY.2, SERVO_RING.2, SERVO_THUMB.2, SERVO_WRIST.2, VREG1.4; no longer S1.2, S2.2, S3.2, S4.2, S5.2, S6.2
- net A0: now also MCU.63; no longer U6.63
- net A1: now also MCU.64; no longer U6.64
- net A2: now also MCU.1; no longer U6.1
- net A3: now also MCU.2; no longer U6.2
- net A4: now also MCU.3; no longer U6.3
- net A5: now also MCU.4; no longer U6.4
- net A6: now also MCU.5; no longer U6.5
- net A7: now also MCU.6; no longer U6.6
- net FSR_INDEX: now also FSR_INDEX.-; no longer FSR4.-
- net FSR_MIDDLE: now also FSR_MIDDLE.-; no longer FSR3.-
- net FSR_PINKY: now also FSR_PINKY.-; no longer FSR1.-
- net FSR_RING: now also FSR_RING.-; no longer FSR2.-
- net FSR_THUMB: now also FSR_THUMB.-; no longer FSR5.-
- net GND: now also MCU.10, MCU.11, MCU.20, MCU.24, MCU.33, MCU.35, MCU.45, MCU.55, MCU.7; no longer C1.2, C10.2, C11.K, C12.2, C13.K, C14.2, C15.K, C16.2, C17.K, C18.2, C2.K, C26.2, C3.2, C4.2, C47.2, C48.2, C49.2, C5.2, C50.2, C51.2, C6.2, C64.2, C7.2, C8.2, C9.K, DEMUX1.12, DEMUX1.15, R16.1, R39.1, R40.1, R41.1, R42.1, S1.3, S2.3, S3.3, S4.3, S5.3, S6.3, TEMP1.3, TEMP2.3, TEMP3.3, TEMP4.3, TEMP5.3, U6.10, U6.11, U6.20, U6.24, U6.33, U6.35, U6.45, U6.55, U6.58, U6.61, U6.7
- net MISO: now also MCU.39; no longer U6.39
- net MOSI: now also MCU.38; no longer U6.38
- net N$30: now also MCU.57; no longer U6.57
- net N$32: now also MCU.9; no longer U6.9
- net N$33: now also MCU.8; no longer U6.8
- net N$35: now also MCU.56; no longer U6.56
- net NGND: now also C1.2, C10.2, C11.K, C12.2, C13.K, C14.2, C15.K, C16.2, C17.K, C2.K, C8.2, C9.K, SERVO_INDEX.3, SERVO_MIDDLE.3, SERVO_PINKY.3, SERVO_RING.3, SERVO_THUMB.3, SERVO_WRIST.3; no longer C85.2, U$2.P$2
- net PB4: now also MCU.40; no longer U6.40
- net PB5: now also MCU.41; no longer U6.41
- net PB6: now also MCU.42; no longer U6.42
- net PB7: now also MCU.43; no longer U6.43
- net PD4: now also MCU.29; no longer U6.29
- net PD5: now also MCU.30; no longer U6.30
- net PD6: now also MCU.31; no longer U6.31
- net PD7: now also MCU.32; no longer U6.32
- net PE2: now also MCU.48; no longer U6.48
- net PE3: now also MCU.49; no longer U6.49
- net PE4: now also MCU.50; no longer U6.50
- net PE5: now also MCU.51; no longer U6.51
- net PE6: now also MCU.52; no longer U6.52
- net PE7: now also MCU.53; no longer U6.53
- net PG0: now also MCU.14; no longer U6.14
- net PG1: now also MCU.15; no longer U6.15
- net PG2: now also MCU.16; no longer U6.16
- net PG3: now also MCU.17; no longer U6.17
- net PG4: now also MCU.18; no longer U6.18
- net PG5: now also MCU.19; no longer U6.19
- net RESET: now also MCU.12; no longer U6.12
- net RX0: now also MCU.46; no longer U6.46
- net RX1: now also MCU.27; no longer U6.27
- net SCK: now also MCU.37; no longer U6.37
- net SCL: now also MCU.25; no longer U6.25
- net SDA: now also MCU.26; no longer U6.26
- net SERVO_INDEX: now also SERVO_INDEX.1; no longer S4.1
- net SERVO_MIDDLE: now also SERVO_MIDDLE.1; no longer S3.1
- net SERVO_PINKY: now also SERVO_PINKY.1; no longer S1.1
- net SERVO_RING: now also SERVO_RING.1; no longer S2.1
- net SERVO_THUMB: now also SERVO_THUMB.1; no longer S5.1
- net SERVO_WRIST: now also SERVO_WRIST.1; no longer S6.1
- net SSN: now also MCU.36; no longer U6.36
- net TEMP_INDEX: now also TEMP_INDEX.2; no longer TEMP4.2
- net TEMP_MIDDLE: now also TEMP_MIDDLE.2; no longer TEMP3.2
- net TEMP_PINKY: now also TEMP_PINKY.2; no longer TEMP1.2
- net TEMP_RING: now also TEMP_RING.2; no longer TEMP2.2
- net TEMP_THUMB: now also TEMP_THUMB.2; no longer TEMP5.2
- net TX0: now also MCU.47; no longer U6.47
- net TX1: now also MCU.28; no longer U6.28
- net VCC: now also MCU.21, MCU.22, MCU.23, MCU.34, MCU.44, MCU.54; no longer C18.1, C26.1, C3.1, C4.1, C47.1, C48.1, C49.1, C5.1, C50.1, C51.1, C56.1, C57.1, C6.1, C64.1, C7.1, C85.1, DEMUX1.24, FSR1.+, FSR2.+, FSR3.+, FSR4.+, FSR5.+, L1.2, TEMP1.1, TEMP2.1, TEMP3.1, TEMP4.1, TEMP5.1, U6.21, U6.22, U6.23, U6.34, U6.44, U6.54, U6.59, U6.60, U6.62
Routing:
- added copper zone on layer 16, net AGND
- added copper zone on layer 1, net GND
Other:
- board size 101.6 x 63.5 mm -> 83.8 x 63.5 mm
- board text added: "RENAME TO GND?"
