File: ecad/electrotactile_extension/electrotactile_extension.sch (EAGLE design)
At the start: 216 parts, among them IC1 DRV8662, J1 VERT MALE 2.54MM, J2 VERT MALE 2.54MM, J3 VERT MALE 2.54MM, J4 VERT MALE 2.54MM, J5 VERT MALE 2.54MM, J6 PTH VERT MALE, J7 PTH VERT MALE, J8 PTH VERT MALE, J9 PTH VERT MALE, SW2 25mA/24V

Commit message: Update work on Electrotactile extension board.  Add doc folder with several schematics breaking down the transmission of touch for documentation purposes.
Parts:
- removed ET_INDEX_PIXEL1-10, ET_INDEX_PIXEL1-11, ET_INDEX_PIXEL1-12, ET_INDEX_PIXEL1-13, ET_INDEX_PIXEL1-14, ET_INDEX_PIXEL1-15, ET_INDEX_PIXEL1-16, ET_INDEX_PIXEL1-17, ET_INDEX_PIXEL1-18, ET_INDEX_PIXEL1-19, ET_INDEX_PIXEL1-20, ET_INDEX_PIXEL1-5, ET_INDEX_PIXEL1-6, ET_INDEX_PIXEL1-7, ET_INDEX_PIXEL1-8, ET_INDEX_PIXEL1-9, ET_INDEX_PIXEL2-10, ET_INDEX_PIXEL2-11, ET_INDEX_PIXEL2-12, ET_INDEX_PIXEL2-13, ET_INDEX_PIXEL2-14, ET_INDEX_PIXEL2-15, ET_INDEX_PIXEL2-16, ET_INDEX_PIXEL2-17, ET_INDEX_PIXEL2-18, ET_INDEX_PIXEL2-19, ET_INDEX_PIXEL2-20, ET_INDEX_PIXEL2-5, ET_INDEX_PIXEL2-6, ET_INDEX_PIXEL2-7, ET_INDEX_PIXEL2-8, ET_INDEX_PIXEL2-9, ET_INDEX_PIXEL3-10, ET_INDEX_PIXEL3-11, ET_INDEX_PIXEL3-12, ET_INDEX_PIXEL3-13, ET_INDEX_PIXEL3-14, ET_INDEX_PIXEL3-15, ET_INDEX_PIXEL3-16, ET_INDEX_PIXEL3-17, ET_INDEX_PIXEL3-18, ET_INDEX_PIXEL3-19, ET_INDEX_PIXEL3-20, ET_INDEX_PIXEL3-5, ET_INDEX_PIXEL3-6, ET_INDEX_PIXEL3-7, ET_INDEX_PIXEL3-8, ET_INDEX_PIXEL3-9, ET_INDEX_PIXEL4-10, ET_INDEX_PIXEL4-11, ET_INDEX_PIXEL4-12, ET_INDEX_PIXEL4-13, ET_INDEX_PIXEL4-14, ET_INDEX_PIXEL4-15, ET_INDEX_PIXEL4-16, ET_INDEX_PIXEL4-17, ET_INDEX_PIXEL4-18, ET_INDEX_PIXEL4-19, ET_INDEX_PIXEL4-20, ET_INDEX_PIXEL4-5, ET_INDEX_PIXEL4-6, ET_INDEX_PIXEL4-7, ET_INDEX_PIXEL4-8, ET_INDEX_PIXEL4-9: SPST-NO 170mA 250V, _relay:RELAY_SOLID-STATE_SSR_170MA_250V_SPST-NO
- removed PWM_DRIVER2, PWM_DRIVER3, PWM_DRIVER4, PWM_DRIVER5, PWM_DRIVER6: PCA9685, _special:PCA9685_16-CH_12-BIT_PWM-DRIVER_TSSOP-28_PWM-DRIVER_16CH
- added ET_MIDDLE_PIXEL1-1, ET_MIDDLE_PIXEL1-2, ET_MIDDLE_PIXEL1-3, ET_MIDDLE_PIXEL1-4, ET_MIDDLE_PIXEL2-1, ET_MIDDLE_PIXEL2-2, ET_MIDDLE_PIXEL2-3, ET_MIDDLE_PIXEL2-4, ET_MIDDLE_PIXEL3-1, ET_MIDDLE_PIXEL3-2, ET_MIDDLE_PIXEL3-3, ET_MIDDLE_PIXEL3-4, ET_MIDDLE_PIXEL4-1, ET_MIDDLE_PIXEL4-2, ET_MIDDLE_PIXEL4-3, ET_MIDDLE_PIXEL4-4, ET_PINKY_PIXEL1-1, ET_PINKY_PIXEL1-2, ET_PINKY_PIXEL1-3, ET_PINKY_PIXEL1-4, ET_PINKY_PIXEL2-1, ET_PINKY_PIXEL2-2, ET_PINKY_PIXEL2-3, ET_PINKY_PIXEL2-4, ET_PINKY_PIXEL3-1, ET_PINKY_PIXEL3-2, ET_PINKY_PIXEL3-3, ET_PINKY_PIXEL3-4, ET_PINKY_PIXEL4-1, ET_PINKY_PIXEL4-2, ET_PINKY_PIXEL4-3, ET_PINKY_PIXEL4-4, ET_RING_PIXEL1-1, ET_RING_PIXEL1-2, ET_RING_PIXEL1-3, ET_RING_PIXEL1-4, ET_RING_PIXEL2-1, ET_RING_PIXEL2-2, ET_RING_PIXEL2-3, ET_RING_PIXEL2-4, ET_RING_PIXEL3-1, ET_RING_PIXEL3-2, ET_RING_PIXEL3-3, ET_RING_PIXEL3-4, ET_RING_PIXEL4-1, ET_RING_PIXEL4-2, ET_RING_PIXEL4-3, ET_RING_PIXEL4-4, ET_THUMB_PIXEL1-1, ET_THUMB_PIXEL1-2, ET_THUMB_PIXEL1-3, ET_THUMB_PIXEL1-4, ET_THUMB_PIXEL2-1, ET_THUMB_PIXEL2-2, ET_THUMB_PIXEL2-3, ET_THUMB_PIXEL2-4, ET_THUMB_PIXEL3-1, ET_THUMB_PIXEL3-2, ET_THUMB_PIXEL3-3, ET_THUMB_PIXEL3-4, ET_THUMB_PIXEL4-1, ET_THUMB_PIXEL4-2, ET_THUMB_PIXEL4-3, ET_THUMB_PIXEL4-4: SPST-NO 170mA 250V, _relay:RELAY_SOLID-STATE_SSR_170MA_250V_SPST-NO
- added MUX_INDEX, MUX_MIDDLE, MUX_PINKY, MUX_RING, MUX_THUMB: PCA9685, _special:PCA9685_16-CH_12-BIT_PWM-DRIVER_TSSOP-28_PWM-DRIVER_16CH
Connections:
- new net MIDDLE_IN1-1: ET_MIDDLE_PIXEL1-1.1, MUX_MIDDLE.PWM14
- new net MIDDLE_IN1-2: ET_MIDDLE_PIXEL1-2.1, MUX_MIDDLE.PWM12
- new net MIDDLE_IN1-3: ET_MIDDLE_PIXEL1-3.1, MUX_MIDDLE.PWM10
- new net MIDDLE_IN1-4: ET_MIDDLE_PIXEL1-4.1, MUX_MIDDLE.PWM8
- new net MIDDLE_IN2-1: ET_MIDDLE_PIXEL2-1.1, MUX_MIDDLE.PWM15
- new net MIDDLE_IN2-2: ET_MIDDLE_PIXEL2-2.1, MUX_MIDDLE.PWM13
- new net MIDDLE_IN2-3: ET_MIDDLE_PIXEL2-3.1, MUX_MIDDLE.PWM11
- new net MIDDLE_IN2-4: ET_MIDDLE_PIXEL2-4.1, MUX_MIDDLE.PWM9
- new net MIDDLE_IN3-1: ET_MIDDLE_PIXEL3-1.1, MUX_MIDDLE.PWM6
- new net MIDDLE_IN3-2: ET_MIDDLE_PIXEL3-2.1, MUX_MIDDLE.PWM4
- new net MIDDLE_IN3-3: ET_MIDDLE_PIXEL3-3.1, MUX_MIDDLE.PWM2
- new net MIDDLE_IN3-4: ET_MIDDLE_PIXEL3-4.1, MUX_MIDDLE.PWM0
- new net MIDDLE_IN4-1: ET_MIDDLE_PIXEL4-1.1, MUX_MIDDLE.PWM7
- new net MIDDLE_IN4-2: ET_MIDDLE_PIXEL4-2.1, MUX_MIDDLE.PWM5
- new net MIDDLE_IN4-3: ET_MIDDLE_PIXEL4-3.1, MUX_MIDDLE.PWM3
- new net MIDDLE_IN4-4: ET_MIDDLE_PIXEL4-4.1, MUX_MIDDLE.PWM1
- new net MIDDLE_OUT1-1: ET_MIDDLE_PIXEL1-1.3
- new net MIDDLE_OUT1-2: ET_MIDDLE_PIXEL1-2.3
- new net MIDDLE_OUT1-3: ET_MIDDLE_PIXEL1-3.3
- new net MIDDLE_OUT1-4: ET_MIDDLE_PIXEL1-4.3
- new net MIDDLE_OUT2-1: ET_MIDDLE_PIXEL2-1.3
- new net MIDDLE_OUT2-2: ET_MIDDLE_PIXEL2-2.3
- new net MIDDLE_OUT2-3: ET_MIDDLE_PIXEL2-3.3
- new net MIDDLE_OUT2-4: ET_MIDDLE_PIXEL2-4.3
- new net MIDDLE_OUT3-1: ET_MIDDLE_PIXEL3-1.3
- new net MIDDLE_OUT3-2: ET_MIDDLE_PIXEL3-2.3
- new net MIDDLE_OUT3-3: ET_MIDDLE_PIXEL3-3.3
- new net MIDDLE_OUT3-4: ET_MIDDLE_PIXEL3-4.3
- new net MIDDLE_OUT4-1: ET_MIDDLE_PIXEL4-1.3
- new net MIDDLE_OUT4-2: ET_MIDDLE_PIXEL4-2.3
- new net MIDDLE_OUT4-3: ET_MIDDLE_PIXEL4-3.3
- new net MIDDLE_OUT4-4: ET_MIDDLE_PIXEL4-4.3
- new net PINKY_IN1-1: ET_PINKY_PIXEL1-1.1, MUX_PINKY.PWM15
- new net PINKY_IN1-2: ET_PINKY_PIXEL1-2.1, MUX_PINKY.PWM13
- new net PINKY_IN1-3: ET_PINKY_PIXEL1-3.1, MUX_PINKY.PWM11
- new net PINKY_IN1-4: ET_PINKY_PIXEL1-4.1, MUX_PINKY.PWM9
- new net PINKY_IN2-1: ET_PINKY_PIXEL2-1.1, MUX_PINKY.PWM14
- new net PINKY_IN2-2: ET_PINKY_PIXEL2-2.1, MUX_PINKY.PWM12
- new net PINKY_IN2-3: ET_PINKY_PIXEL2-3.1, MUX_PINKY.PWM10
- new net PINKY_IN2-4: ET_PINKY_PIXEL2-4.1, MUX_PINKY.PWM8
- new net PINKY_IN3-1: ET_PINKY_PIXEL3-1.1, MUX_PINKY.PWM7
- new net PINKY_IN3-2: ET_PINKY_PIXEL3-2.1, MUX_PINKY.PWM5
- new net PINKY_IN3-3: ET_PINKY_PIXEL3-3.1, MUX_PINKY.PWM3
- new net PINKY_IN3-4: ET_PINKY_PIXEL3-4.1, MUX_PINKY.PWM1
- new net PINKY_IN4-1: ET_PINKY_PIXEL4-1.1, MUX_PINKY.PWM6
- new net PINKY_IN4-2: ET_PINKY_PIXEL4-2.1, MUX_PINKY.PWM4
- new net PINKY_IN4-3: ET_PINKY_PIXEL4-3.1, MUX_PINKY.PWM2
- new net PINKY_IN4-4: ET_PINKY_PIXEL4-4.1, MUX_PINKY.PWM0
- new net PINKY_OUT1-1: ET_PINKY_PIXEL1-1.3
- new net PINKY_OUT1-2: ET_PINKY_PIXEL1-2.3
- new net PINKY_OUT1-3: ET_PINKY_PIXEL1-3.3
- new net PINKY_OUT1-4: ET_PINKY_PIXEL1-4.3
- new net PINKY_OUT2-1: ET_PINKY_PIXEL2-1.3
- new net PINKY_OUT2-2: ET_PINKY_PIXEL2-2.3
- new net PINKY_OUT2-3: ET_PINKY_PIXEL2-3.3
- new net PINKY_OUT2-4: ET_PINKY_PIXEL2-4.3
- new net PINKY_OUT3-1: ET_PINKY_PIXEL3-1.3
- new net PINKY_OUT3-2: ET_PINKY_PIXEL3-2.3
- new net PINKY_OUT3-3: ET_PINKY_PIXEL3-3.3
- new net PINKY_OUT3-4: ET_PINKY_PIXEL3-4.3
- new net PINKY_OUT4-1: ET_PINKY_PIXEL4-1.3
- new net PINKY_OUT4-2: ET_PINKY_PIXEL4-2.3
- new net PINKY_OUT4-3: ET_PINKY_PIXEL4-3.3
- new net PINKY_OUT4-4: ET_PINKY_PIXEL4-4.3
- new net RING_IN1-1: ET_RING_PIXEL1-1.1, MUX_RING.PWM1
- new net RING_IN1-2: ET_RING_PIXEL1-2.1, MUX_RING.PWM3
- new net RING_IN1-3: ET_RING_PIXEL1-3.1, MUX_RING.PWM5
- new net RING_IN1-4: ET_RING_PIXEL1-4.1, MUX_RING.PWM7
- new net RING_IN2-1: ET_RING_PIXEL2-1.1, MUX_RING.PWM0
- new net RING_IN2-2: ET_RING_PIXEL2-2.1, MUX_RING.PWM2
- new net RING_IN2-3: ET_RING_PIXEL2-3.1, MUX_RING.PWM4
- new net RING_IN2-4: ET_RING_PIXEL2-4.1, MUX_RING.PWM6
- new net RING_IN3-1: ET_RING_PIXEL3-1.1, MUX_RING.PWM9
- new net RING_IN3-2: ET_RING_PIXEL3-2.1, MUX_RING.PWM11
- new net RING_IN3-3: ET_RING_PIXEL3-3.1, MUX_RING.PWM13
- new net RING_IN3-4: ET_RING_PIXEL3-4.1, MUX_RING.PWM15
- new net RING_IN4-1: ET_RING_PIXEL4-1.1, MUX_RING.PWM8
- new net RING_IN4-2: ET_RING_PIXEL4-2.1, MUX_RING.PWM10
- new net RING_IN4-3: ET_RING_PIXEL4-3.1, MUX_RING.PWM12
- new net RING_IN4-4: ET_RING_PIXEL4-4.1, MUX_RING.PWM14
- new net RING_OUT1-1: ET_RING_PIXEL1-1.3
- new net RING_OUT1-2: ET_RING_PIXEL1-2.3
- new net RING_OUT1-3: ET_RING_PIXEL1-3.3
- new net RING_OUT1-4: ET_RING_PIXEL1-4.3
- new net RING_OUT2-1: ET_RING_PIXEL2-1.3
- new net RING_OUT2-2: ET_RING_PIXEL2-2.3
- new net RING_OUT2-3: ET_RING_PIXEL2-3.3
- new net RING_OUT2-4: ET_RING_PIXEL2-4.3
- new net RING_OUT3-1: ET_RING_PIXEL3-1.3
- new net RING_OUT3-2: ET_RING_PIXEL3-2.3
- new net RING_OUT3-3: ET_RING_PIXEL3-3.3
- new net RING_OUT3-4: ET_RING_PIXEL3-4.3
- new net RING_OUT4-1: ET_RING_PIXEL4-1.3
- new net RING_OUT4-2: ET_RING_PIXEL4-2.3
- new net RING_OUT4-3: ET_RING_PIXEL4-3.3
- new net RING_OUT4-4: ET_RING_PIXEL4-4.3
- new net THUMB_IN1-1: ET_THUMB_PIXEL1-1.1, MUX_THUMB.PWM0
- new net THUMB_IN1-2: ET_THUMB_PIXEL1-2.1, MUX_THUMB.PWM1
- new net THUMB_IN1-3: ET_THUMB_PIXEL1-3.1, MUX_THUMB.PWM2
- new net THUMB_IN1-4: ET_THUMB_PIXEL1-4.1, MUX_THUMB.PWM3
- new net THUMB_IN2-1: ET_THUMB_PIXEL2-1.1, MUX_THUMB.PWM4
- new net THUMB_IN2-2: ET_THUMB_PIXEL2-2.1, MUX_THUMB.PWM5
- new net THUMB_IN2-3: ET_THUMB_PIXEL2-3.1, MUX_THUMB.PWM6
- new net THUMB_IN2-4: ET_THUMB_PIXEL2-4.1, MUX_THUMB.PWM7
- new net THUMB_IN3-1: ET_THUMB_PIXEL3-1.1, MUX_THUMB.PWM8
- new net THUMB_IN3-2: ET_THUMB_PIXEL3-2.1, MUX_THUMB.PWM9
- new net THUMB_IN3-3: ET_THUMB_PIXEL3-3.1, MUX_THUMB.PWM10
- new net THUMB_IN3-4: ET_THUMB_PIXEL3-4.1, MUX_THUMB.PWM11
- new net THUMB_IN4-1: ET_THUMB_PIXEL4-1.1, MUX_THUMB.PWM12
- new net THUMB_IN4-2: ET_THUMB_PIXEL4-2.1, MUX_THUMB.PWM13
- new net THUMB_IN4-3: ET_THUMB_PIXEL4-3.1, MUX_THUMB.PWM14
- new net THUMB_IN4-4: ET_THUMB_PIXEL4-4.1, MUX_THUMB.PWM15
- new net THUMB_OUT1-1: ET_THUMB_PIXEL1-1.3
- new net THUMB_OUT1-2: ET_THUMB_PIXEL1-2.3
- new net THUMB_OUT1-3: ET_THUMB_PIXEL1-3.3
- new net THUMB_OUT1-4: ET_THUMB_PIXEL1-4.3
- new net THUMB_OUT2-1: ET_THUMB_PIXEL2-1.3
- new net THUMB_OUT2-2: ET_THUMB_PIXEL2-2.3
- new net THUMB_OUT2-3: ET_THUMB_PIXEL2-3.3
- new net THUMB_OUT2-4: ET_THUMB_PIXEL2-4.3
- new net THUMB_OUT3-1: ET_THUMB_PIXEL3-1.3
- new net THUMB_OUT3-2: ET_THUMB_PIXEL3-2.3
- new net THUMB_OUT3-3: ET_THUMB_PIXEL3-3.3
- new net THUMB_OUT3-4: ET_THUMB_PIXEL3-4.3
- new net THUMB_OUT4-1: ET_THUMB_PIXEL4-1.3
- new net THUMB_OUT4-2: ET_THUMB_PIXEL4-2.3
- new net THUMB_OUT4-3: ET_THUMB_PIXEL4-3.3
- new net THUMB_OUT4-4: ET_THUMB_PIXEL4-4.3
- net GND: now also MUX_INDEX.!OE, MUX_INDEX.A0, MUX_INDEX.A1, MUX_INDEX.A2, MUX_INDEX.A3, MUX_INDEX.A4, MUX_INDEX.A5, MUX_INDEX.EXTCLK, MUX_INDEX.GND, MUX_MIDDLE.!OE, MUX_MIDDLE.A0, MUX_MIDDLE.A1, MUX_MIDDLE.A2, MUX_MIDDLE.A3, MUX_MIDDLE.A4, MUX_MIDDLE.A5, MUX_MIDDLE.EXTCLK, MUX_MIDDLE.GND, MUX_PINKY.!OE, MUX_PINKY.A0, MUX_PINKY.A1, MUX_PINKY.A2, MUX_PINKY.A3, MUX_PINKY.A4, MUX_PINKY.A5, MUX_PINKY.EXTCLK, MUX_PINKY.GND, MUX_RING.!OE, MUX_RING.A0, MUX_RING.A1, MUX_RING.A2, MUX_RING.A3, MUX_RING.A4, MUX_RING.A5, MUX_RING.EXTCLK, MUX_RING.GND, MUX_THUMB.!OE, MUX_THUMB.A0, MUX_THUMB.A1, MUX_THUMB.A2, MUX_THUMB.A3, MUX_THUMB.A4, MUX_THUMB.A5, MUX_THUMB.EXTCLK, MUX_THUMB.GND; no longer PWM_DRIVER2.!OE, PWM_DRIVER2.A0, PWM_DRIVER2.A1, PWM_DRIVER2.A2, PWM_DRIVER2.A3, PWM_DRIVER2.A4, PWM_DRIVER2.A5, PWM_DRIVER2.EXTCLK, PWM_DRIVER2.GND, PWM_DRIVER3.!OE, PWM_DRIVER3.A0, PWM_DRIVER3.A1, PWM_DRIVER3.A2, PWM_DRIVER3.A3, PWM_DRIVER3.A4, PWM_DRIVER3.A5, PWM_DRIVER3.EXTCLK, PWM_DRIVER3.GND, PWM_DRIVER4.!OE, PWM_DRIVER4.A0, PWM_DRIVER4.A1, PWM_DRIVER4.A2, PWM_DRIVER4.A3, PWM_DRIVER4.A4, PWM_DRIVER4.A5, PWM_DRIVER4.EXTCLK, PWM_DRIVER4.GND, PWM_DRIVER5.!OE, PWM_DRIVER5.A0, PWM_DRIVER5.A1, PWM_DRIVER5.A2, PWM_DRIVER5.A3, PWM_DRIVER5.A4, PWM_DRIVER5.A5, PWM_DRIVER5.EXTCLK, PWM_DRIVER5.GND, PWM_DRIVER6.!OE, PWM_DRIVER6.A0, PWM_DRIVER6.A1, PWM_DRIVER6.A2, PWM_DRIVER6.A3, PWM_DRIVER6.A4, PWM_DRIVER6.A5, PWM_DRIVER6.EXTCLK, PWM_DRIVER6.GND
- net INDEX_IN1-1: now also MUX_INDEX.PWM0; no longer ET_INDEX_PIXEL1-13.1, ET_INDEX_PIXEL1-17.1, ET_INDEX_PIXEL1-5.1, ET_INDEX_PIXEL1-9.1, PWM_DRIVER2.PWM0, PWM_DRIVER3.PWM0, PWM_DRIVER4.PWM0, PWM_DRIVER5.PWM0, PWM_DRIVER6.PWM0
- net INDEX_IN1-2: now also MUX_INDEX.PWM2; no longer ET_INDEX_PIXEL1-10.1, ET_INDEX_PIXEL1-14.1, ET_INDEX_PIXEL1-18.1, ET_INDEX_PIXEL1-6.1, PWM_DRIVER2.PWM1, PWM_DRIVER3.PWM1, PWM_DRIVER4.PWM1, PWM_DRIVER5.PWM1, PWM_DRIVER6.PWM1
- net INDEX_IN1-3: now also MUX_INDEX.PWM4; no longer ET_INDEX_PIXEL1-11.1, ET_INDEX_PIXEL1-15.1, ET_INDEX_PIXEL1-19.1, ET_INDEX_PIXEL1-7.1, PWM_DRIVER2.PWM2, PWM_DRIVER3.PWM2, PWM_DRIVER4.PWM2, PWM_DRIVER5.PWM2, PWM_DRIVER6.PWM2
- net INDEX_IN1-4: now also MUX_INDEX.PWM6; no longer ET_INDEX_PIXEL1-12.1, ET_INDEX_PIXEL1-16.1, ET_INDEX_PIXEL1-20.1, ET_INDEX_PIXEL1-8.1, PWM_DRIVER2.PWM3, PWM_DRIVER3.PWM3, PWM_DRIVER4.PWM3, PWM_DRIVER5.PWM3, PWM_DRIVER6.PWM3
- net INDEX_IN2-1: now also MUX_INDEX.PWM1; no longer ET_INDEX_PIXEL2-11.1, ET_INDEX_PIXEL2-15.1, ET_INDEX_PIXEL2-19.1, ET_INDEX_PIXEL2-7.1, PWM_DRIVER2.PWM4, PWM_DRIVER3.PWM4, PWM_DRIVER4.PWM4, PWM_DRIVER5.PWM4, PWM_DRIVER6.PWM4
- net INDEX_IN2-2: now also MUX_INDEX.PWM3; no longer ET_INDEX_PIXEL2-10.1, ET_INDEX_PIXEL2-14.1, ET_INDEX_PIXEL2-18.1, ET_INDEX_PIXEL2-6.1, PWM_DRIVER2.PWM5, PWM_DRIVER3.PWM5, PWM_DRIVER4.PWM5, PWM_DRIVER5.PWM5, PWM_DRIVER6.PWM5
- net INDEX_IN2-3: now also MUX_INDEX.PWM5; no longer ET_INDEX_PIXEL2-13.1, ET_INDEX_PIXEL2-17.1, ET_INDEX_PIXEL2-5.1, ET_INDEX_PIXEL2-9.1, PWM_DRIVER2.PWM6, PWM_DRIVER3.PWM6, PWM_DRIVER4.PWM6, PWM_DRIVER5.PWM6, PWM_DRIVER6.PWM6
- net INDEX_IN2-4: now also MUX_INDEX.PWM7; no longer ET_INDEX_PIXEL2-12.1, ET_INDEX_PIXEL2-16.1, ET_INDEX_PIXEL2-20.1, ET_INDEX_PIXEL2-8.1, PWM_DRIVER2.PWM7, PWM_DRIVER3.PWM7, PWM_DRIVER4.PWM7, PWM_DRIVER5.PWM7, PWM_DRIVER6.PWM7
- net INDEX_IN3-1: now also MUX_INDEX.PWM8; no longer ET_INDEX_PIXEL3-13.1, ET_INDEX_PIXEL3-17.1, ET_INDEX_PIXEL3-5.1, ET_INDEX_PIXEL3-9.1, PWM_DRIVER2.PWM8, PWM_DRIVER3.PWM8, PWM_DRIVER4.PWM8, PWM_DRIVER5.PWM8, PWM_DRIVER6.PWM8
- net INDEX_IN3-2: now also MUX_INDEX.PWM10; no longer ET_INDEX_PIXEL3-10.1, ET_INDEX_PIXEL3-14.1, ET_INDEX_PIXEL3-18.1, ET_INDEX_PIXEL3-6.1, PWM_DRIVER2.PWM9, PWM_DRIVER3.PWM9, PWM_DRIVER4.PWM9, PWM_DRIVER5.PWM9, PWM_DRIVER6.PWM9
- net INDEX_IN3-3: now also MUX_INDEX.PWM12; no longer ET_INDEX_PIXEL3-11.1, ET_INDEX_PIXEL3-15.1, ET_INDEX_PIXEL3-19.1, ET_INDEX_PIXEL3-7.1, PWM_DRIVER2.PWM10, PWM_DRIVER3.PWM10, PWM_DRIVER4.PWM10, PWM_DRIVER5.PWM10, PWM_DRIVER6.PWM10
- net INDEX_IN3-4: now also MUX_INDEX.PWM14; no longer ET_INDEX_PIXEL3-12.1, ET_INDEX_PIXEL3-16.1, ET_INDEX_PIXEL3-20.1, ET_INDEX_PIXEL3-8.1, PWM_DRIVER2.PWM11, PWM_DRIVER3.PWM11, PWM_DRIVER4.PWM11, PWM_DRIVER5.PWM11, PWM_DRIVER6.PWM11
- net INDEX_IN4-1: now also MUX_INDEX.PWM9; no longer ET_INDEX_PIXEL4-13.1, ET_INDEX_PIXEL4-17.1, ET_INDEX_PIXEL4-5.1, ET_INDEX_PIXEL4-9.1, PWM_DRIVER2.PWM12, PWM_DRIVER3.PWM12, PWM_DRIVER4.PWM12, PWM_DRIVER5.PWM12, PWM_DRIVER6.PWM12
- net INDEX_IN4-2: now also MUX_INDEX.PWM11; no longer ET_INDEX_PIXEL4-10.1, ET_INDEX_PIXEL4-14.1, ET_INDEX_PIXEL4-18.1, ET_INDEX_PIXEL4-6.1, PWM_DRIVER2.PWM13, PWM_DRIVER3.PWM13, PWM_DRIVER4.PWM13, PWM_DRIVER5.PWM13, PWM_DRIVER6.PWM13
- net INDEX_IN4-3: now also MUX_INDEX.PWM13; no longer ET_INDEX_PIXEL4-11.1, ET_INDEX_PIXEL4-15.1, ET_INDEX_PIXEL4-19.1, ET_INDEX_PIXEL4-7.1, PWM_DRIVER2.PWM14, PWM_DRIVER3.PWM14, PWM_DRIVER4.PWM14, PWM_DRIVER5.PWM14, PWM_DRIVER6.PWM14
- net INDEX_IN4-4: now also MUX_INDEX.PWM15; no longer ET_INDEX_PIXEL4-12.1, ET_INDEX_PIXEL4-16.1, ET_INDEX_PIXEL4-20.1, ET_INDEX_PIXEL4-8.1, PWM_DRIVER2.PWM15, PWM_DRIVER3.PWM15, PWM_DRIVER4.PWM15, PWM_DRIVER5.PWM15, PWM_DRIVER6.PWM15
- net INDEX_OUT1-1: no longer ET_INDEX_PIXEL1-13.3, ET_INDEX_PIXEL1-17.3, ET_INDEX_PIXEL1-5.3, ET_INDEX_PIXEL1-9.3
- net INDEX_OUT1-2: no longer ET_INDEX_PIXEL1-10.3, ET_INDEX_PIXEL1-14.3, ET_INDEX_PIXEL1-18.3, ET_INDEX_PIXEL1-6.3
- net INDEX_OUT1-3: no longer ET_INDEX_PIXEL1-11.3, ET_INDEX_PIXEL1-15.3, ET_INDEX_PIXEL1-19.3, ET_INDEX_PIXEL1-7.3
- net INDEX_OUT1-4: no longer ET_INDEX_PIXEL1-12.3, ET_INDEX_PIXEL1-16.3, ET_INDEX_PIXEL1-20.3, ET_INDEX_PIXEL1-8.3
- net INDEX_OUT2-1: no longer ET_INDEX_PIXEL2-11.3, ET_INDEX_PIXEL2-15.3, ET_INDEX_PIXEL2-19.3, ET_INDEX_PIXEL2-7.3
- net INDEX_OUT2-2: no longer ET_INDEX_PIXEL2-10.3, ET_INDEX_PIXEL2-14.3, ET_INDEX_PIXEL2-18.3, ET_INDEX_PIXEL2-6.3
- net INDEX_OUT2-3: no longer ET_INDEX_PIXEL2-13.3, ET_INDEX_PIXEL2-17.3, ET_INDEX_PIXEL2-5.3, ET_INDEX_PIXEL2-9.3
- net INDEX_OUT2-4: no longer ET_INDEX_PIXEL2-12.3, ET_INDEX_PIXEL2-16.3, ET_INDEX_PIXEL2-20.3, ET_INDEX_PIXEL2-8.3
- net INDEX_OUT3-1: no longer ET_INDEX_PIXEL3-13.3, ET_INDEX_PIXEL3-17.3, ET_INDEX_PIXEL3-5.3, ET_INDEX_PIXEL3-9.3
- net INDEX_OUT3-2: no longer ET_INDEX_PIXEL3-10.3, ET_INDEX_PIXEL3-14.3, ET_INDEX_PIXEL3-18.3, ET_INDEX_PIXEL3-6.3
- net INDEX_OUT3-3: no longer ET_INDEX_PIXEL3-11.3, ET_INDEX_PIXEL3-15.3, ET_INDEX_PIXEL3-19.3, ET_INDEX_PIXEL3-7.3
- net INDEX_OUT3-4: no longer ET_INDEX_PIXEL3-12.3, ET_INDEX_PIXEL3-16.3, ET_INDEX_PIXEL3-20.3, ET_INDEX_PIXEL3-8.3
- net INDEX_OUT4-1: no longer ET_INDEX_PIXEL4-13.3, ET_INDEX_PIXEL4-17.3, ET_INDEX_PIXEL4-5.3, ET_INDEX_PIXEL4-9.3
- net INDEX_OUT4-2: no longer ET_INDEX_PIXEL4-10.3, ET_INDEX_PIXEL4-14.3, ET_INDEX_PIXEL4-18.3, ET_INDEX_PIXEL4-6.3
- net INDEX_OUT4-3: no longer ET_INDEX_PIXEL4-11.3, ET_INDEX_PIXEL4-15.3, ET_INDEX_PIXEL4-19.3, ET_INDEX_PIXEL4-7.3
- net INDEX_OUT4-4: no longer ET_INDEX_PIXEL4-12.3, ET_INDEX_PIXEL4-16.3, ET_INDEX_PIXEL4-20.3, ET_INDEX_PIXEL4-8.3
- net N$100: now also ET_MIDDLE_PIXEL3-4.2; no longer ET_INDEX_PIXEL3-12.2
- net N$101: now also ET_MIDDLE_PIXEL4-1.2; no longer ET_INDEX_PIXEL4-9.2
- net N$102: now also ET_MIDDLE_PIXEL4-2.2; no longer ET_INDEX_PIXEL4-10.2
- net N$103: now also ET_MIDDLE_PIXEL4-3.2; no longer ET_INDEX_PIXEL4-11.2
- net N$104: now also ET_MIDDLE_PIXEL4-4.2; no longer ET_INDEX_PIXEL4-12.2
- net N$105: now also ET_RING_PIXEL1-1.2; no longer ET_INDEX_PIXEL1-13.2
- net N$106: now also ET_RING_PIXEL1-2.2; no longer ET_INDEX_PIXEL1-14.2
- net N$107: now also ET_RING_PIXEL1-3.2; no longer ET_INDEX_PIXEL1-15.2
- net N$108: now also ET_RING_PIXEL1-4.2; no longer ET_INDEX_PIXEL1-16.2
- net N$109: now also ET_RING_PIXEL2-1.2; no longer ET_INDEX_PIXEL2-15.2
- net N$110: now also ET_RING_PIXEL2-2.2; no longer ET_INDEX_PIXEL2-14.2
- net N$111: now also ET_RING_PIXEL2-3.2; no longer ET_INDEX_PIXEL2-13.2
- net N$112: now also ET_RING_PIXEL2-4.2; no longer ET_INDEX_PIXEL2-16.2
- net N$113: now also ET_RING_PIXEL3-1.2; no longer ET_INDEX_PIXEL3-13.2
- net N$114: now also ET_RING_PIXEL3-2.2; no longer ET_INDEX_PIXEL3-14.2
- net N$115: now also ET_RING_PIXEL3-3.2; no longer ET_INDEX_PIXEL3-15.2
- net N$116: now also ET_RING_PIXEL3-4.2; no longer ET_INDEX_PIXEL3-16.2
- net N$117: now also ET_RING_PIXEL4-1.2; no longer ET_INDEX_PIXEL4-13.2
- net N$118: now also ET_RING_PIXEL4-2.2; no longer ET_INDEX_PIXEL4-14.2
- net N$119: now also ET_RING_PIXEL4-3.2; no longer ET_INDEX_PIXEL4-15.2
- net N$120: now also ET_RING_PIXEL4-4.2; no longer ET_INDEX_PIXEL4-16.2
- net N$121: now also ET_PINKY_PIXEL1-1.2; no longer ET_INDEX_PIXEL1-17.2
- net N$122: now also ET_PINKY_PIXEL1-2.2; no longer ET_INDEX_PIXEL1-18.2
- net N$123: now also ET_PINKY_PIXEL1-3.2; no longer ET_INDEX_PIXEL1-19.2
- net N$124: now also ET_PINKY_PIXEL1-4.2; no longer ET_INDEX_PIXEL1-20.2
- net N$125: now also ET_PINKY_PIXEL2-1.2; no longer ET_INDEX_PIXEL2-19.2
- net N$126: now also ET_PINKY_PIXEL2-2.2; no longer ET_INDEX_PIXEL2-18.2
- net N$127: now also ET_PINKY_PIXEL2-3.2; no longer ET_INDEX_PIXEL2-17.2
- net N$128: now also ET_PINKY_PIXEL2-4.2; no longer ET_INDEX_PIXEL2-20.2
- net N$129: now also ET_PINKY_PIXEL3-1.2; no longer ET_INDEX_PIXEL3-17.2
- net N$130: now also ET_PINKY_PIXEL3-2.2; no longer ET_INDEX_PIXEL3-18.2
- net N$131: now also ET_PINKY_PIXEL3-3.2; no longer ET_INDEX_PIXEL3-19.2
- net N$132: now also ET_PINKY_PIXEL3-4.2; no longer ET_INDEX_PIXEL3-20.2
- net N$133: now also ET_PINKY_PIXEL4-1.2; no longer ET_INDEX_PIXEL4-17.2
- net N$134: now also ET_PINKY_PIXEL4-2.2; no longer ET_INDEX_PIXEL4-18.2
- net N$135: now also ET_PINKY_PIXEL4-3.2; no longer ET_INDEX_PIXEL4-19.2
- net N$136: now also ET_PINKY_PIXEL4-4.2; no longer ET_INDEX_PIXEL4-20.2
- net N$58: now also ET_THUMB_PIXEL1-1.2; no longer ET_INDEX_PIXEL1-5.2
- net N$74: now also ET_THUMB_PIXEL1-2.2; no longer ET_INDEX_PIXEL1-6.2
- net N$75: now also ET_THUMB_PIXEL1-3.2; no longer ET_INDEX_PIXEL1-7.2
- net N$76: now also ET_THUMB_PIXEL1-4.2; no longer ET_INDEX_PIXEL1-8.2
- net N$77: now also ET_THUMB_PIXEL2-1.2; no longer ET_INDEX_PIXEL2-7.2
- net N$78: now also ET_THUMB_PIXEL2-2.2; no longer ET_INDEX_PIXEL2-6.2
- net N$79: now also ET_THUMB_PIXEL2-3.2; no longer ET_INDEX_PIXEL2-5.2
- net N$80: now also ET_THUMB_PIXEL2-4.2; no longer ET_INDEX_PIXEL2-8.2
- net N$81: now also ET_THUMB_PIXEL3-1.2; no longer ET_INDEX_PIXEL3-5.2
- net N$82: now also ET_THUMB_PIXEL3-2.2; no longer ET_INDEX_PIXEL3-6.2
- net N$83: now also ET_THUMB_PIXEL3-3.2; no longer ET_INDEX_PIXEL3-7.2
- net N$84: now also ET_THUMB_PIXEL3-4.2; no longer ET_INDEX_PIXEL3-8.2
- net N$85: now also ET_THUMB_PIXEL4-1.2; no longer ET_INDEX_PIXEL4-5.2
- net N$86: now also ET_THUMB_PIXEL4-2.2; no longer ET_INDEX_PIXEL4-6.2
- net N$87: now also ET_THUMB_PIXEL4-3.2; no longer ET_INDEX_PIXEL4-7.2
- net N$88: now also ET_THUMB_PIXEL4-4.2; no longer ET_INDEX_PIXEL4-8.2
- net N$89: now also ET_MIDDLE_PIXEL1-1.2; no longer ET_INDEX_PIXEL1-9.2
- net N$90: now also ET_MIDDLE_PIXEL1-2.2; no longer ET_INDEX_PIXEL1-10.2
- net N$91: now also ET_MIDDLE_PIXEL1-3.2; no longer ET_INDEX_PIXEL1-11.2
- net N$92: now also ET_MIDDLE_PIXEL1-4.2; no longer ET_INDEX_PIXEL1-12.2
- net N$93: now also ET_MIDDLE_PIXEL2-1.2; no longer ET_INDEX_PIXEL2-11.2
- net N$94: now also ET_MIDDLE_PIXEL2-2.2; no longer ET_INDEX_PIXEL2-10.2
- net N$95: now also ET_MIDDLE_PIXEL2-3.2; no longer ET_INDEX_PIXEL2-9.2
- net N$96: now also ET_MIDDLE_PIXEL2-4.2; no longer ET_INDEX_PIXEL2-12.2
- net N$97: now also ET_MIDDLE_PIXEL3-1.2; no longer ET_INDEX_PIXEL3-9.2
- net N$98: now also ET_MIDDLE_PIXEL3-2.2; no longer ET_INDEX_PIXEL3-10.2
- net N$99: now also ET_MIDDLE_PIXEL3-3.2; no longer ET_INDEX_PIXEL3-11.2
- net SCL: now also MUX_INDEX.SCL, MUX_MIDDLE.SCL, MUX_PINKY.SCL, MUX_RING.SCL, MUX_THUMB.SCL; no longer PWM_DRIVER2.SCL, PWM_DRIVER3.SCL, PWM_DRIVER4.SCL, PWM_DRIVER5.SCL, PWM_DRIVER6.SCL
- net SDA: now also MUX_INDEX.SDA, MUX_MIDDLE.SDA, MUX_PINKY.SDA, MUX_RING.SDA, MUX_THUMB.SDA; no longer PWM_DRIVER2.SDA, PWM_DRIVER3.SDA, PWM_DRIVER4.SDA, PWM_DRIVER5.SDA, PWM_DRIVER6.SDA
- net V+: now also ET_MIDDLE_PIXEL1-1.4, ET_MIDDLE_PIXEL1-2.4, ET_MIDDLE_PIXEL1-3.4, ET_MIDDLE_PIXEL1-4.4, ET_MIDDLE_PIXEL2-1.4, ET_MIDDLE_PIXEL2-2.4, ET_MIDDLE_PIXEL2-3.4, ET_MIDDLE_PIXEL2-4.4, ET_MIDDLE_PIXEL3-1.4, ET_MIDDLE_PIXEL3-2.4, ET_MIDDLE_PIXEL3-3.4, ET_MIDDLE_PIXEL3-4.4, ET_MIDDLE_PIXEL4-1.4, ET_MIDDLE_PIXEL4-2.4, ET_MIDDLE_PIXEL4-3.4, ET_MIDDLE_PIXEL4-4.4, ET_PINKY_PIXEL1-1.4, ET_PINKY_PIXEL1-2.4, ET_PINKY_PIXEL1-3.4, ET_PINKY_PIXEL1-4.4, ET_PINKY_PIXEL2-1.4, ET_PINKY_PIXEL2-2.4, ET_PINKY_PIXEL2-3.4, ET_PINKY_PIXEL2-4.4, ET_PINKY_PIXEL3-1.4, ET_PINKY_PIXEL3-2.4, ET_PINKY_PIXEL3-3.4, ET_PINKY_PIXEL3-4.4, ET_PINKY_PIXEL4-1.4, ET_PINKY_PIXEL4-2.4, ET_PINKY_PIXEL4-3.4, ET_PINKY_PIXEL4-4.4, ET_RING_PIXEL1-1.4, ET_RING_PIXEL1-2.4, ET_RING_PIXEL1-3.4, ET_RING_PIXEL1-4.4, ET_RING_PIXEL2-1.4, ET_RING_PIXEL2-2.4, ET_RING_PIXEL2-3.4, ET_RING_PIXEL2-4.4, ET_RING_PIXEL3-1.4, ET_RING_PIXEL3-2.4, ET_RING_PIXEL3-3.4, ET_RING_PIXEL3-4.4, ET_RING_PIXEL4-1.4, ET_RING_PIXEL4-2.4, ET_RING_PIXEL4-3.4, ET_RING_PIXEL4-4.4, ET_THUMB_PIXEL1-1.4, ET_THUMB_PIXEL1-2.4, ET_THUMB_PIXEL1-3.4, ET_THUMB_PIXEL1-4.4, ET_THUMB_PIXEL2-1.4, ET_THUMB_PIXEL2-2.4, ET_THUMB_PIXEL2-3.4, ET_THUMB_PIXEL2-4.4, ET_THUMB_PIXEL3-1.4, ET_THUMB_PIXEL3-2.4, ET_THUMB_PIXEL3-3.4, ET_THUMB_PIXEL3-4.4, ET_THUMB_PIXEL4-1.4, ET_THUMB_PIXEL4-2.4, ET_THUMB_PIXEL4-3.4, ET_THUMB_PIXEL4-4.4; no longer ET_INDEX_PIXEL1-10.4, ET_INDEX_PIXEL1-11.4, ET_INDEX_PIXEL1-12.4, ET_INDEX_PIXEL1-13.4, ET_INDEX_PIXEL1-14.4, ET_INDEX_PIXEL1-15.4, ET_INDEX_PIXEL1-16.4, ET_INDEX_PIXEL1-17.4, ET_INDEX_PIXEL1-18.4, ET_INDEX_PIXEL1-19.4, ET_INDEX_PIXEL1-20.4, ET_INDEX_PIXEL1-5.4, ET_INDEX_PIXEL1-6.4, ET_INDEX_PIXEL1-7.4, ET_INDEX_PIXEL1-8.4, ET_INDEX_PIXEL1-9.4, ET_INDEX_PIXEL2-10.4, ET_INDEX_PIXEL2-11.4, ET_INDEX_PIXEL2-12.4, ET_INDEX_PIXEL2-13.4, ET_INDEX_PIXEL2-14.4, ET_INDEX_PIXEL2-15.4, ET_INDEX_PIXEL2-16.4, ET_INDEX_PIXEL2-17.4, ET_INDEX_PIXEL2-18.4, ET_INDEX_PIXEL2-19.4, ET_INDEX_PIXEL2-20.4, ET_INDEX_PIXEL2-5.4, ET_INDEX_PIXEL2-6.4, ET_INDEX_PIXEL2-7.4, ET_INDEX_PIXEL2-8.4, ET_INDEX_PIXEL2-9.4, ET_INDEX_PIXEL3-10.4, ET_INDEX_PIXEL3-11.4, ET_INDEX_PIXEL3-12.4, ET_INDEX_PIXEL3-13.4, ET_INDEX_PIXEL3-14.4, ET_INDEX_PIXEL3-15.4, ET_INDEX_PIXEL3-16.4, ET_INDEX_PIXEL3-17.4, ET_INDEX_PIXEL3-18.4, ET_INDEX_PIXEL3-19.4, ET_INDEX_PIXEL3-20.4, ET_INDEX_PIXEL3-5.4, ET_INDEX_PIXEL3-6.4, ET_INDEX_PIXEL3-7.4, ET_INDEX_PIXEL3-8.4, ET_INDEX_PIXEL3-9.4, ET_INDEX_PIXEL4-10.4, ET_INDEX_PIXEL4-11.4, ET_INDEX_PIXEL4-12.4, ET_INDEX_PIXEL4-13.4, ET_INDEX_PIXEL4-14.4, ET_INDEX_PIXEL4-15.4, ET_INDEX_PIXEL4-16.4, ET_INDEX_PIXEL4-17.4, ET_INDEX_PIXEL4-18.4, ET_INDEX_PIXEL4-19.4, ET_INDEX_PIXEL4-20.4, ET_INDEX_PIXEL4-5.4, ET_INDEX_PIXEL4-6.4, ET_INDEX_PIXEL4-7.4, ET_INDEX_PIXEL4-8.4, ET_INDEX_PIXEL4-9.4
- net VCC: now also MUX_INDEX.VCC, MUX_MIDDLE.VCC, MUX_PINKY.VCC, MUX_RING.VCC, MUX_THUMB.VCC; no longer PWM_DRIVER2.VCC, PWM_DRIVER3.VCC, PWM_DRIVER4.VCC, PWM_DRIVER5.VCC, PWM_DRIVER6.VCC
Other:
- moved on the sheet: C37, C49, C61, C62, C63, C64, C65, C66, C67, C68, C69, C70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

Commit message: Create PCA9685Servo library.  Touch up Touch Glove PCB.  Major work completed on ET Extension.
Parts:
- removed C67: 0.1uF/50V, _capacitors:0.1UF_SMD-0402_50V-10%
- removed ET_THUMB_PIXEL1-1, ET_THUMB_PIXEL1-2, ET_THUMB_PIXEL1-3, ET_THUMB_PIXEL1-4, ET_THUMB_PIXEL2-1, ET_THUMB_PIXEL2-2, ET_THUMB_PIXEL2-3, ET_THUMB_PIXEL2-4, ET_THUMB_PIXEL3-1, ET_THUMB_PIXEL3-2, ET_THUMB_PIXEL3-3, ET_THUMB_PIXEL3-4, ET_THUMB_PIXEL4-1, ET_THUMB_PIXEL4-2, ET_THUMB_PIXEL4-3, ET_THUMB_PIXEL4-4: SPST-NO 170mA 250V, _relay:RELAY_SOLID-STATE_SSR_170MA_250V_SPST-NO
- removed J2: VERT MALE 2.54MM, _connectors:1X16_PTH_VERT_MALE_2.54MM
- removed MUX_THUMB: PCA9685, _special:PCA9685_16-CH_12-BIT_PWM-DRIVER_TSSOP-28_PWM-DRIVER_16CH
- removed R72, R73, R74, R75, R76, R77, R78, R79, R80, R81, R82, R83, R84, R85, R86, R87: 1K, _resistors:1KΩ_SMD-0402_1/16W-5%
- removed SW2: 25mA/24V, _switches:SWITCH_SPST_ARRAY-3_SLIDE_DIP_SPST_25MA_24V
- added SW1, SW3, SW4: 300mA/4V, _switches:SWITCH_SPDT_RA_SMD_300MA-4V_6.7L-2.6W
Connections:
- removed net N$58: ET_THUMB_PIXEL1-1.2, R72.2
- removed net N$7: VREG3.EN
- removed net N$74: ET_THUMB_PIXEL1-2.2, R73.2
- removed net N$75: ET_THUMB_PIXEL1-3.2, R74.2
- removed net N$76: ET_THUMB_PIXEL1-4.2, R75.2
- removed net N$77: ET_THUMB_PIXEL2-1.2, R76.2
- removed net N$78: ET_THUMB_PIXEL2-2.2, R77.2
- removed net N$79: ET_THUMB_PIXEL2-3.2, R78.2
- removed net N$80: ET_THUMB_PIXEL2-4.2, R79.2
- removed net N$81: ET_THUMB_PIXEL3-1.2, R80.2
- removed net N$82: ET_THUMB_PIXEL3-2.2, R81.2
- removed net N$83: ET_THUMB_PIXEL3-3.2, R82.2
- removed net N$84: ET_THUMB_PIXEL3-4.2, R83.2
- removed net N$85: ET_THUMB_PIXEL4-1.2, R84.2
- removed net N$86: ET_THUMB_PIXEL4-2.2, R85.2
- removed net N$87: ET_THUMB_PIXEL4-3.2, R86.2
- removed net N$88: ET_THUMB_PIXEL4-4.2, R87.2
- removed net NGND: J8.1, J8.2
- removed net THUMB_IN1-1: ET_THUMB_PIXEL1-1.1, MUX_THUMB.PWM0
- removed net THUMB_IN1-2: ET_THUMB_PIXEL1-2.1, MUX_THUMB.PWM1
- removed net THUMB_IN1-3: ET_THUMB_PIXEL1-3.1, MUX_THUMB.PWM2
- removed net THUMB_IN1-4: ET_THUMB_PIXEL1-4.1, MUX_THUMB.PWM3
- removed net THUMB_IN2-1: ET_THUMB_PIXEL2-1.1, MUX_THUMB.PWM4
- removed net THUMB_IN2-2: ET_THUMB_PIXEL2-2.1, MUX_THUMB.PWM5
- removed net THUMB_IN2-3: ET_THUMB_PIXEL2-3.1, MUX_THUMB.PWM6
- removed net THUMB_IN2-4: ET_THUMB_PIXEL2-4.1, MUX_THUMB.PWM7
- removed net THUMB_IN3-1: ET_THUMB_PIXEL3-1.1, MUX_THUMB.PWM8
- removed net THUMB_IN3-2: ET_THUMB_PIXEL3-2.1, MUX_THUMB.PWM9
- removed net THUMB_IN3-3: ET_THUMB_PIXEL3-3.1, MUX_THUMB.PWM10
- removed net THUMB_IN3-4: ET_THUMB_PIXEL3-4.1, MUX_THUMB.PWM11
- removed net THUMB_IN4-1: ET_THUMB_PIXEL4-1.1, MUX_THUMB.PWM12
- removed net THUMB_IN4-2: ET_THUMB_PIXEL4-2.1, MUX_THUMB.PWM13
- removed net THUMB_IN4-3: ET_THUMB_PIXEL4-3.1, MUX_THUMB.PWM14
- removed net THUMB_IN4-4: ET_THUMB_PIXEL4-4.1, MUX_THUMB.PWM15
- removed net THUMB_OUT1-1: ET_THUMB_PIXEL1-1.3
- removed net THUMB_OUT1-2: ET_THUMB_PIXEL1-2.3
- removed net THUMB_OUT1-3: ET_THUMB_PIXEL1-3.3
- removed net THUMB_OUT1-4: ET_THUMB_PIXEL1-4.3
- removed net THUMB_OUT2-1: ET_THUMB_PIXEL2-1.3
- removed net THUMB_OUT2-2: ET_THUMB_PIXEL2-2.3
- removed net THUMB_OUT2-3: ET_THUMB_PIXEL2-3.3
- removed net THUMB_OUT2-4: ET_THUMB_PIXEL2-4.3
- removed net THUMB_OUT3-1: ET_THUMB_PIXEL3-1.3
- removed net THUMB_OUT3-2: ET_THUMB_PIXEL3-2.3
- removed net THUMB_OUT3-3: ET_THUMB_PIXEL3-3.3
- removed net THUMB_OUT3-4: ET_THUMB_PIXEL3-4.3
- removed net THUMB_OUT4-1: ET_THUMB_PIXEL4-1.3
- removed net THUMB_OUT4-2: ET_THUMB_PIXEL4-2.3
- removed net THUMB_OUT4-3: ET_THUMB_PIXEL4-3.3
- removed net THUMB_OUT4-4: ET_THUMB_PIXEL4-4.3
- removed net VCC: C66.1, C67.1, C68.1, C69.1, C70.1, MUX_INDEX.VCC, MUX_MIDDLE.VCC, MUX_PINKY.VCC, MUX_RING.VCC, MUX_THUMB.VCC
- net 3.3V: now also C66.1, C68.1, C69.1, C70.1, MUX_INDEX.A1, MUX_INDEX.VCC, MUX_MIDDLE.A0, MUX_MIDDLE.A1, MUX_MIDDLE.VCC, MUX_PINKY.A0, MUX_PINKY.A2, MUX_PINKY.VCC, MUX_RING.A2, MUX_RING.VCC, SW1.P, SW3.P, SW4.P, VREG3.EN; no longer SW2.P1, SW2.P2, SW2.P3
- net EN: now also SW1.S2; no longer SW2.S3
- net GAIN0: now also SW3.S2; no longer SW2.S2
- net GAIN1: now also SW4.S2; no longer SW2.S1
- net GND: no longer C67.2, MUX_INDEX.A1, MUX_MIDDLE.A0, MUX_MIDDLE.A1, MUX_PINKY.A0, MUX_PINKY.A2, MUX_RING.A2, MUX_THUMB.!OE, MUX_THUMB.A0, MUX_THUMB.A1, MUX_THUMB.A2, MUX_THUMB.A3, MUX_THUMB.A4, MUX_THUMB.A5, MUX_THUMB.EXTCLK, MUX_THUMB.GND, R72.1, R73.1, R74.1, R75.1, R76.1, R77.1, R78.1, R79.1, R80.1, R81.1, R82.1, R83.1, R84.1, R85.1, R86.1, R87.1
- net INDEX_OUT1-1: no longer J2.1
- net SCL: no longer MUX_THUMB.SCL
- net SDA: no longer MUX_THUMB.SDA
- net V+: no longer ET_THUMB_PIXEL1-1.4, ET_THUMB_PIXEL1-2.4, ET_THUMB_PIXEL1-3.4, ET_THUMB_PIXEL1-4.4, ET_THUMB_PIXEL2-1.4, ET_THUMB_PIXEL2-2.4, ET_THUMB_PIXEL2-3.4, ET_THUMB_PIXEL2-4.4, ET_THUMB_PIXEL3-1.4, ET_THUMB_PIXEL3-2.4, ET_THUMB_PIXEL3-3.4, ET_THUMB_PIXEL3-4.4, ET_THUMB_PIXEL4-1.4, ET_THUMB_PIXEL4-2.4, ET_THUMB_PIXEL4-3.4, ET_THUMB_PIXEL4-4.4
- net V-: no longer J2.16
Other:
- note added: "+1.8V VREG"
- note added: "+3.3V VREG"
- note added: "-1.8V VREG"
- note added: "0x42"
- note added: "0x43"
- note added: "0x44"
- note added: "0x45"
- note removed: "ET ARRAY - THUMB"
- note removed: "NC"
- note removed: "TODO: Change I2C addr"
- note removed: "TODO: NAME ENABLE PIN"
- moved on the sheet: C71, C72, C73, C74, C75, C76, C77, C78, C79, C80, L4, OPAMP4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

Commit message: Complete iteration of ET Extension and Touch Glove.  Verify PCA9685Servo library works and made appropriate changes in robotic arm master code.
Parts:
- removed J1, J3, J4, J5: VERT MALE 2.54MM, _connectors:1X16_PTH_VERT_MALE_2.54MM
- added INDEX_CONNECTOR, MIDDLE_CONNECTOR, PINKY_CONNECTOR, RING_CONNECTOR: 1x17 MOLEX SMD RA, _connectors:1X17_SMD_MOLEX
- J6, J7, J8, J9: value PTH VERT MALE -> 1x02 PTH VERT FEMALE; device _connectors:1X02_PTH_VERT_MALE_2.54MM -> _connectors:1X02_PTH_VERT_FEMALE_2.54MM
Connections:
- net INDEX_OUT1-1: now also INDEX_CONNECTOR.1; no longer J1.1, J3.1, J4.1, J5.1
- net INDEX_OUT1-2: now also INDEX_CONNECTOR.3
- net INDEX_OUT1-3: now also INDEX_CONNECTOR.5
- net INDEX_OUT1-4: now also INDEX_CONNECTOR.7
- net INDEX_OUT2-1: now also INDEX_CONNECTOR.2
- net INDEX_OUT2-2: now also INDEX_CONNECTOR.4
- net INDEX_OUT2-3: now also INDEX_CONNECTOR.6
- net INDEX_OUT2-4: now also INDEX_CONNECTOR.8
- net INDEX_OUT3-1: now also INDEX_CONNECTOR.9
- net INDEX_OUT3-2: now also INDEX_CONNECTOR.11
- net INDEX_OUT3-3: now also INDEX_CONNECTOR.13
- net INDEX_OUT3-4: now also INDEX_CONNECTOR.15
- net INDEX_OUT4-1: now also INDEX_CONNECTOR.10
- net INDEX_OUT4-2: now also INDEX_CONNECTOR.12
- net INDEX_OUT4-3: now also INDEX_CONNECTOR.14
- net INDEX_OUT4-4: now also INDEX_CONNECTOR.16
- net MIDDLE_OUT1-1: now also MIDDLE_CONNECTOR.16
- net MIDDLE_OUT1-2: now also MIDDLE_CONNECTOR.14
- net MIDDLE_OUT1-3: now also MIDDLE_CONNECTOR.12
- net MIDDLE_OUT1-4: now also MIDDLE_CONNECTOR.10
- net MIDDLE_OUT2-1: now also MIDDLE_CONNECTOR.17
- net MIDDLE_OUT2-2: now also MIDDLE_CONNECTOR.15
- net MIDDLE_OUT2-3: now also MIDDLE_CONNECTOR.13
- net MIDDLE_OUT2-4: now also MIDDLE_CONNECTOR.11
- net MIDDLE_OUT3-1: now also MIDDLE_CONNECTOR.8
- net MIDDLE_OUT3-2: now also MIDDLE_CONNECTOR.6
- net MIDDLE_OUT3-3: now also MIDDLE_CONNECTOR.4
- net MIDDLE_OUT3-4: now also MIDDLE_CONNECTOR.2
- net MIDDLE_OUT4-1: now also MIDDLE_CONNECTOR.9
- net MIDDLE_OUT4-2: now also MIDDLE_CONNECTOR.7
- net MIDDLE_OUT4-3: now also MIDDLE_CONNECTOR.5
- net MIDDLE_OUT4-4: now also MIDDLE_CONNECTOR.3
- net PINKY_OUT1-1: now also PINKY_CONNECTOR.16
- net PINKY_OUT1-2: now also PINKY_CONNECTOR.14
- net PINKY_OUT1-3: now also PINKY_CONNECTOR.12
- net PINKY_OUT1-4: now also PINKY_CONNECTOR.10
- net PINKY_OUT2-1: now also PINKY_CONNECTOR.17
- net PINKY_OUT2-2: now also PINKY_CONNECTOR.15
- net PINKY_OUT2-3: now also PINKY_CONNECTOR.13
- net PINKY_OUT2-4: now also PINKY_CONNECTOR.11
- net PINKY_OUT3-1: now also PINKY_CONNECTOR.8
- net PINKY_OUT3-2: now also PINKY_CONNECTOR.6
- net PINKY_OUT3-3: now also PINKY_CONNECTOR.4
- net PINKY_OUT3-4: now also PINKY_CONNECTOR.2
- net PINKY_OUT4-1: now also PINKY_CONNECTOR.9
- net PINKY_OUT4-2: now also PINKY_CONNECTOR.7
- net PINKY_OUT4-3: now also PINKY_CONNECTOR.5
- net PINKY_OUT4-4: now also PINKY_CONNECTOR.3
- net RING_OUT1-1: now also RING_CONNECTOR.1
- net RING_OUT1-2: now also RING_CONNECTOR.3
- net RING_OUT1-3: now also RING_CONNECTOR.5
- net RING_OUT1-4: now also RING_CONNECTOR.7
- net RING_OUT2-1: now also RING_CONNECTOR.2
- net RING_OUT2-2: now also RING_CONNECTOR.4
- net RING_OUT2-3: now also RING_CONNECTOR.6
- net RING_OUT2-4: now also RING_CONNECTOR.8
- net RING_OUT3-1: now also RING_CONNECTOR.9
- net RING_OUT3-2: now also RING_CONNECTOR.11
- net RING_OUT3-3: now also RING_CONNECTOR.13
- net RING_OUT3-4: now also RING_CONNECTOR.15
- net RING_OUT4-1: now also RING_CONNECTOR.10
- net RING_OUT4-2: now also RING_CONNECTOR.12
- net RING_OUT4-3: now also RING_CONNECTOR.14
- net RING_OUT4-4: now also RING_CONNECTOR.16
- net V-: now also INDEX_CONNECTOR.17, MIDDLE_CONNECTOR.1, PINKY_CONNECTOR.1, RING_CONNECTOR.17; no longer J1.16, J3.16, J4.16, J5.16
Other:
- moved on the sheet: C66, C68, C69, C70, ET_INDEX_PIXEL1-1, ET_INDEX_PIXEL1-2, ET_INDEX_PIXEL1-3, ET_INDEX_PIXEL1-4, ET_INDEX_PIXEL2-1, ET_INDEX_PIXEL2-2, ET_INDEX_PIXEL2-3, ET_INDEX_PIXEL2-4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

Commit message: Lots of changes.  But rip.
Parts:
- C61: value 0.1uF/25V -> 0.1uF/50V
- C62: value 0.1uF/250V -> 0.1uF/250V/0805
- L3: value 4.7uH/1.4A -> 4.7uH/2A/1008; device _inductors:4.7UH_SMD-2520_1.4A-0.216OHM-20% -> _inductors:4.7UH_SMD-1008_2A-0.200OHM-20%
Changed lines of the file:
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@@
 <part name="C49" library="_capacitors" deviceset="0.1UF" device="_SMD-0402_50V-10%" package3d_urn="urn:adsk.eagle:package:2886515/1" value="0.1uF/50V"/>
 <part name="SUPPLY132" library="_power_symbols" deviceset="GND" device=""/>
-<part name="L3" library="_inductors" deviceset="4.7UH" device="_SMD-2520_1.4A-0.216OHM-20%" package3d_urn="urn:adsk.eagle:package:6898949/1" value="4.7uH/1.4A"/>
-<part name="C61" library="_capacitors" deviceset="0.1UF" device="_SMD-0603_50V-20%" package3d_urn="urn:adsk.eagle:package:3041595/1" value="0.1uF/25V"/>
+<part name="L3" library="_inductors" deviceset="4.7UH" device="_SMD-1008_2A-0.200OHM-20%" package3d_urn="urn:adsk.eagle:package:6898949/1" value="4.7uH/2A/1008"/>
+<part name="C61" library="_capacitors" deviceset="0.1UF" device="_SMD-0603_50V-20%" package3d_urn="urn:adsk.eagle:package:3041595/1" value="0.1uF/50V"/>
 <part name="SUPPLY133" library="_power_symbols" deviceset="GND" device=""/>
 <part name="R50" library="_resistors" deviceset="768KΩ" device="_SMD-0402_1/16W-1%" package3d_urn="urn:adsk.eagle:package:2899165/1" value="768K"/>
-<part name="C62" library="_capacitors" deviceset="0.1UF" device="_SMD-0805_250V-10%" package3d_urn="urn:adsk.eagle:package:2940050/1" value="0.1uF/250V"/>
+<part name="C62" library="_capacitors" deviceset="0.1UF" device="_SMD-0805_250V-10%" package3d_urn="urn:adsk.eagle:package:2940050/1" value="0.1uF/250V/0805"/>
 <part name="SUPPLY135" library="_power_symbols" deviceset="GND" device=""/>
 <part name="NFET1" library="_transistors" deviceset="MOSFET_N-CHANNEL_2-ARRAY" device="_2N7002DW_115MA-60V" package3d_urn="urn:adsk.eagle:package:6899146/1" value="2N7002DW"/>

Commit message: Everything fucking works (have not tested ET driver extensively yet though)
Other:
- note removed: "TODO: CHECK VALUES (C1, POT1, R2,R3) AND VOLTAGE DIVIDER TO MAKE 1.8V"
- note removed: "Transfer: VBAT, SDA, SCL, GND"
Changed lines of the file:
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@@
 <wire x1="657.86" y1="195.58" x2="657.86" y2="325.12" width="0.1524" layer="97" style="shortdash"/>
 <text x="482.6" y="327.66" size="5.08" layer="97" font="vector" ratio="20" align="bottom-center">ET ARRAY - PINKY</text>
-<text x="68.58" y="711.2" size="1.778" layer="91" rot="R180">TODO: CHECK VALUES (C1, POT1, R2,R3) AND VOLTAGE DIVIDER TO MAKE 1.8V</text>
 <wire x1="55.88" y1="701.04" x2="55.88" y2="764.54" width="0.1524" layer="97" style="shortdash"/>
 <wire x1="111.76" y1="701.04" x2="55.88" y2="701.04" width="0.1524" layer="97" style="shortdash"/>
@@
 <text x="185.42" y="792.48" size="1.778" layer="91">STAGE2</text>
 <text x="472.44" y="800.1" size="1.778" layer="91">STAGE3</text>
-<text x="0" y="668.02" size="1.778" layer="91">Transfer: VBAT, SDA, SCL, GND</text>
 <wire x1="-152.4" y1="728.98" x2="-88.9" y2="728.98" width="0.1524" layer="97" style="shortdash"/>
 <wire x1="-88.9" y1="728.98" x2="-88.9" y2="764.54" width="0.1524" layer="97" style="shortdash"/>
