File: ecad/robotic_arm/robotic_arm.brd (EAGLE design)
At the start: 59.7 x 57.9 mm, 112 parts, among them J1 5A/28V, SW1 5A/28V, Y1 16 MHz

Commit message: Lots of changes.  But rip.
Parts:
- C61: value 22pF/100V -> 22pF/100V/0402
Changed lines of the file:
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@@
 <attribute name="VALUE" x="35.5" y="47.1" size="0.5" layer="27" font="vector" ratio="10" align="top-center"/>
 </element>
-<element name="C61" library="_capacitors" package="CAPC1005X55_SMD-0402" package3d_urn="urn:adsk.eagle:package:2886515/1" value="22pF/100V" x="32.87" y="48.176" smashed="yes" rot="R180">
-<attribute name="DATASHEET" value="http://ds.yuden.co.jp/TYCOMPAS/ut/detail.do?productNo=HMK105CG220JV-F&amp;fileName=HMK105CG220JV-F_SS&amp;mode=specSheetDownload" x="557.634" y="272.712" size="1.778" layer="27" rot="R180" display="off"/>
+<element name="C61" library="_capacitors" package="CAPC1005X55_SMD-0402" package3d_urn="urn:adsk.eagle:package:2886515/1" value="22pF/100V/0402" x="32.87" y="48.176" smashed="yes" rot="R180">
+<attribute name="DATASHEET" value="http://www.vishay.com/docs/45071/vjhifreq.pdf" x="557.634" y="272.712" size="1.778" layer="27" rot="R180" display="off"/>
 <attribute name="DIST" value="Digikey" x="557.634" y="272.712" size="1.778" layer="27" rot="R180" display="off"/>
-<attribute name="DISTLINK" value="https://www.digikey.com/products/en?keywords=587-5004-1-ND" x="557.634" y="272.712" size="1.778" layer="27" rot="R180" display="off"/>
-<attribute name="DISTPN" value="587-5004-1-ND" x="557.634" y="272.712" size="1.778" layer="27" rot="R180" display="off"/>
-<attribute name="MFR" value="Taiyo Yuden" x="557.634" y="272.712" size="1.778" layer="27" rot="R180" display="off"/>
-<attribute name="MPN" value="HMK105CG220JV-F" x="557.634" y="272.712" size="1.778" layer="27" rot="R180" display="off"/>
+<attribute name="DISTLINK" value="https://www.digikey.com/products/en?keywords=720-1286-1-ND" x="557.634" y="272.712" size="1.778" layer="27" rot="R180" display="off"/>
+<attribute name="DISTPN" value="720-1286-1-ND" x="557.634" y="272.712" size="1.778" layer="27" rot="R180" display="off"/>
+<attribute name="MFR" value="Vishay Vitramon" x="557.634" y="272.712" size="1.778" layer="27" rot="R180" display="off"/>
+<attribute name="MPN" value="VJ0402D220JXBAJ" x="557.634" y="272.712" size="1.778" layer="27" rot="R180" display="off"/>
 <attribute name="NAME" x="32.87" y="47.541" size="0.5" layer="25" font="vector" ratio="10" rot="R180" align="bottom-center"/>
-<attribute name="VALUE" x="32.87" y="48.811" size="0.25" layer="27" font="vector" ratio="10" rot="R180" align="top-center"/>
+<attribute name="VALUE" value="22pF/100V/0402" x="32.87" y="48.811" size="0.25" layer="27" font="vector" ratio="10" rot="R180" align="top-center"/>
 </element>
 <element name="C62" library="_capacitors" package="CAPC1005X55_SMD-0402" package3d_urn="urn:adsk.eagle:package:2886515/1" value="0.75pF/50V" x="32.87" y="49.412" smashed="yes" rot="R180">
@@
 <attribute name="MPN" value="CDSQR4148-HF" x="28.3" y="46.8" size="1.778" layer="27" rot="R180" display="off"/>
 <attribute name="NAME" x="28.3" y="46.1" size="0.5" layer="25" font="vector" ratio="10" rot="R180" align="bottom-center"/>
-<attribute name="VALUE" x="28.3" y="47.5" size="0.5" layer="27" font="vector" ratio="10" rot="R180" align="top-center"/>
+<attribute name="VALUE" x="28.3" y="47.5" size="0.25" layer="27" font="vector" ratio="10" rot="R180" align="top-center"/>
 </element>
 <element name="NOISE_BR" library="_power_symbols" package="NET_BRIDGE" value="NET_BRIDGE" x="28.3" y="7.9" smashed="yes" rot="MR180"/>

Commit message: Everything fucking works (have not tested ET driver extensively yet though)
Parts:
- moved FSR_PINKY 17.8 mm to (52.5, 15.1)
- moved FSR_THUMB 17.8 mm to (52.5, 32.9)
- moved FSR_INDEX 8.90 mm to (52.5, 28.4)
- moved FSR_RING 8.90 mm to (52.5, 19.5)
Connections:
- net FSR_INDEX: now also FSR_INDEX.2; no longer FSR_RING.2
- net FSR_PINKY: now also FSR_PINKY.2; no longer FSR_THUMB.2
- net FSR_RING: now also FSR_RING.2; no longer FSR_INDEX.2
- net FSR_THUMB: now also FSR_THUMB.2; no longer FSR_PINKY.2
Changed lines of the file:
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@@
 </layers>
 <board>
-<fusionsync huburn="a.cGVyc29uYWw6dWUyOTIwMzJm" projecturn="a.cGVyc29uYWw6dWUyOTIwMzJmIzIwMTgwNTE1MTMyMDQwMDA2" f3durn="urn:adsk.wipprod:dm.lineage:j3vuE3OiS_mCt6szVSR7Aw" pcbguid="7ab83d0f-2879-46d5-9d19-329c08f3fa45" lastpulledtime="" lastsyncedchangeguid="da6dde38-6ba1-632f-1d2d-d1609a38c80a"/>
+<fusionsync huburn="a.cGVyc29uYWw6dWUyOTIwMzJm" projecturn="a.cGVyc29uYWw6dWUyOTIwMzJmIzIwMTgwNTE1MTMyMDQwMDA2" f3durn="urn:adsk.wipprod:dm.lineage:j3vuE3OiS_mCt6szVSR7Aw" pcbguid="7ab83d0f-2879-46d5-9d19-329c08f3fa45" lastpulledtime="" lastsyncedchangeguid="3b90e577-0645-c454-68ff-a75af2f08b4f"/>
 <plain>
 <wire x1="0" y1="57.9" x2="0" y2="0" width="0" layer="20"/>
@@
 <attribute name="VALUE" value="TPS76833QDR 1A/3.3V" x="36.1" y="25.633" size="0.25" layer="27" font="vector" ratio="10" align="top-center"/>
 </element>
-<element name="FSR_PINKY" library="_sensors" package="_MOLEX-0530470210_VERT_PITCH-1.25MM" package3d_urn="urn:adsk.eagle:package:2973718/2" value="10K" x="52.55" y="32.85" smashed="yes" rot="R270">
+<element name="FSR_THUMB" library="_sensors" package="_MOLEX-0530470210_VERT_PITCH-1.25MM" package3d_urn="urn:adsk.eagle:package:2973718/2" value="10K" x="52.55" y="32.85" smashed="yes" rot="R270">
 <attribute name="DATASHEET" value="https://cdn2.hubspot.net/hubfs/3899023/Interlinkelectronics%20November2017/Docs/Datasheet_FSR.pdf" x="52.55" y="32.85" size="1.778" layer="27" rot="R270" display="off"/>
 <attribute name="DATASHEET_CONNECTOR1" value="https://www.molex.com/pdm_docs/sd/530470210_sd.pdf" x="52.55" y="32.85" size="1.778" layer="27" rot="R270" display="off"/>
@@
 <attribute name="VALUE" x="53.185" y="32.85" size="0.25" layer="27" font="vector" ratio="10" rot="R270" align="bottom-center"/>
 </element>
-<element name="FSR_RING" library="_sensors" package="_MOLEX-0530470210_VERT_PITCH-1.25MM" package3d_urn="urn:adsk.eagle:package:2973718/2" value="10K" x="52.55" y="28.4" smashed="yes" rot="R270">
+<element name="FSR_INDEX" library="_sensors" package="_MOLEX-0530470210_VERT_PITCH-1.25MM" package3d_urn="urn:adsk.eagle:package:2973718/2" value="10K" x="52.55" y="28.4" smashed="yes" rot="R270">
 <attribute name="DATASHEET" value="https://cdn2.hubspot.net/hubfs/3899023/Interlinkelectronics%20November2017/Docs/Datasheet_FSR.pdf" x="52.55" y="28.4" size="1.778" layer="27" rot="R270" display="off"/>
 <attribute name="DATASHEET_CONNECTOR1" value="https://www.molex.com/pdm_docs/sd/530470210_sd.pdf" x="52.55" y="28.4" size="1.778" layer="27" rot="R270" display="off"/>
@@
 <attribute name="VALUE" x="53.185" y="23.95" size="0.25" layer="27" font="vector" ratio="10" rot="R270" align="bottom-center"/>
 </element>
-<element name="FSR_INDEX" library="_sensors" package="_MOLEX-0530470210_VERT_PITCH-1.25MM" package3d_urn="urn:adsk.eagle:package:2973718/2" value="10K" x="52.55" y="19.5" smashed="yes" rot="R270">
+<element name="FSR_RING" library="_sensors" package="_MOLEX-0530470210_VERT_PITCH-1.25MM" package3d_urn="urn:adsk.eagle:package:2973718/2" value="10K" x="52.55" y="19.5" smashed="yes" rot="R270">
 <attribute name="DATASHEET" value="https://cdn2.hubspot.net/hubfs/3899023/Interlinkelectronics%20November2017/Docs/Datasheet_FSR.pdf" x="52.55" y="19.5" size="1.778" layer="27" rot="R270" display="off"/>
 <attribute name="DATASHEET_CONNECTOR1" value="https://www.molex.com/pdm_docs/sd/530470210_sd.pdf" x="52.55" y="19.5" size="1.778" layer="27" rot="R270" display="off"/>
@@
 <attribute name="VALUE" x="53.185" y="19.5" size="0.25" layer="27" font="vector" ratio="10" rot="R270" align="bottom-center"/>
 </element>
-<element name="FSR_THUMB" library="_sensors" package="_MOLEX-0530470210_VERT_PITCH-1.25MM" package3d_urn="urn:adsk.eagle:package:2973718/2" value="10K" x="52.55" y="15.05" smashed="yes" rot="R270">
+<element name="FSR_PINKY" library="_sensors" package="_MOLEX-0530470210_VERT_PITCH-1.25MM" package3d_urn="urn:adsk.eagle:package:2973718/2" value="10K" x="52.55" y="15.05" smashed="yes" rot="R270">
 <attribute name="DATASHEET" value="https://cdn2.hubspot.net/hubfs/3899023/Interlinkelectronics%20November2017/Docs/Datasheet_FSR.pdf" x="52.55" y="15.05" size="1.778" layer="27" rot="R270" display="off"/>
 <attribute name="DATASHEET_CONNECTOR1" value="https://www.molex.com/pdm_docs/sd/530470210_sd.pdf" x="52.55" y="15.05" size="1.778" layer="27" rot="R270" display="off"/>
@@
 <signal name="FSR_PINKY">
 <contactref element="R42" pad="2"/>
-<contactref element="FSR_THUMB" pad="2"/>
+<contactref element="FSR_PINKY" pad="2"/>
 <wire x1="50.7325" y1="14.4" x2="52.525" y2="14.4" width="0.1524" layer="1"/>
 <wire x1="52.525" y1="14.4" x2="52.55" y2="14.425" width="0.1524" layer="1"/>
@@
 <signal name="FSR_RING">
 <contactref element="R41" pad="2"/>
-<contactref element="FSR_INDEX" pad="2"/>
+<contactref element="FSR_RING" pad="2"/>
 <wire x1="52.55" y1="18.875" x2="52.525" y2="18.9" width="0.1524" layer="1"/>
 <wire x1="52.525" y1="18.9" x2="50.7325" y2="18.9" width="0.1524" layer="1"/>
@@
 <signal name="FSR_INDEX">
 <contactref element="R39" pad="2"/>
-<contactref element="FSR_RING" pad="2"/>
+<contactref element="FSR_INDEX" pad="2"/>
 <wire x1="50.7325" y1="27.75" x2="52.525" y2="27.75" width="0.1524" layer="1"/>
 <wire x1="52.525" y1="27.75" x2="52.55" y2="27.775" width="0.1524" layer="1"/>
@@
 <signal name="FSR_THUMB">
 <contactref element="R16" pad="2"/>
-<contactref element="FSR_PINKY" pad="2"/>
+<contactref element="FSR_THUMB" pad="2"/>
 <wire x1="50.7325" y1="32.2" x2="52.525" y2="32.2" width="0.1524" layer="1"/>
 <wire x1="52.525" y1="32.2" x2="52.55" y2="32.225" width="0.1524" layer="1"/>
@@
 <signal name="VSENSOR">
 <contactref element="JP3" pad="2"/>
-<contactref element="FSR_PINKY" pad="1"/>
+<contactref element="FSR_THUMB" pad="1"/>
 <contactref element="C47" pad="1"/>
-<contactref element="FSR_RING" pad="1"/>
+<contactref element="FSR_INDEX" pad="1"/>
 <contactref element="FSR_MIDDLE" pad="1"/>
 <contactref element="C49" pad="1"/>
-<contactref element="FSR_INDEX" pad="1"/>
+<contactref element="FSR_RING" pad="1"/>
 <contactref element="C50" pad="1"/>
-<contactref element="FSR_THUMB" pad="1"/>
+<contactref element="FSR_PINKY" pad="1"/>
 <contactref element="C51" pad="1"/>
 <contactref element="C48" pad="1"/>
