File: ecad/robotic_arm/robotic_arm.sch (EAGLE design)
At the start: 108 parts, among them J1 5A/28V, SW1 5A/28V, Y1 16 MHz

Commit message: Create PCA9685Servo library.  Update robotic arm PCB to Rev 3.  Ready for fab.
Parts:
- C11, C13, C15, C17, C9: device _capacitors:100UF-POLARIZED_SMD_25V-20%_DIA5-LS2-H11 -> _capacitors:100UF-POLARIZED_PTH_25V-20%_D5-LS2-H11
- C20, C27, C80: device _capacitors:1000UF-POLARIZED_PTH_16V-20% -> _capacitors:1000UF-POLARIZED_PTH_16V-20%_D8-LS3.5-H20
Changed lines of the file:
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@@
 <?xml version="1.0" encoding="utf-8"?>
 <!DOCTYPE eagle SYSTEM "eagle.dtd">
-<eagle version="9.3.0">
+<eagle version="9.3.1">
 <drawing>
 <settings>
@@
 <part name="GND124" library="_power_symbols" deviceset="GND" device=""/>
 <part name="NGND1" library="_power_symbols" deviceset="NGND" device="" value="NGND"/>
-<part name="SW1" library="_switches" deviceset="SWITCH_SPDT" device="_VERT_PTH_5A-28V_13L-7W_" package3d_urn="urn:adsk.eagle:package:3033359/4" value="5A/28V"/>
 <part name="GND125" library="_power_symbols" deviceset="GND" device=""/>
 <part name="D7" library="_discrete_semiconductors" deviceset="GENERAL-PURPOSE" device="_SMD_GP_1A-50V" package3d_urn="urn:adsk.eagle:package:2939213/1" value="1A/50V"/>
-<part name="C80" library="_capacitors" deviceset="1000UF-POLARIZED" device="_PTH_16V-20%" package3d_urn="urn:adsk.eagle:package:3036236/2" value="1000uF/16V"/>
+<part name="C80" library="_capacitors" deviceset="1000UF-POLARIZED" device="_PTH_16V-20%_D8-LS3.5-H20" package3d_urn="urn:adsk.eagle:package:9488079/1" value="1000uF/16V"/>
 <part name="GND127" library="_power_symbols" deviceset="GND" device=""/>
 <part name="L1" library="_inductors" deviceset="10UH" device="_SMD-0603_0.38A-0.468OHM-10%" package3d_urn="urn:adsk.eagle:package:2899745/1" value="10uH/380mA"/>
@@
 <part name="C21" library="_capacitors" deviceset="1UF" device="_CER_SMD-0402_25V-10%" package3d_urn="urn:adsk.eagle:package:2886515/1" value="1uF/25V"/>
 <part name="GND17" library="_power_symbols" deviceset="GND" device=""/>
-<part name="C20" library="_capacitors" deviceset="1000UF-POLARIZED" device="_PTH_16V-20%" package3d_urn="urn:adsk.eagle:package:3036236/2" value="1000uF/16V"/>
+<part name="C20" library="_capacitors" deviceset="1000UF-POLARIZED" device="_PTH_16V-20%_D8-LS3.5-H20" package3d_urn="urn:adsk.eagle:package:9488079/1" value="1000uF/16V"/>
 <part name="C23" library="_capacitors" deviceset="1UF" device="_CER_SMD-0402_25V-10%" package3d_urn="urn:adsk.eagle:package:2886515/1" value="1uF/25V"/>
 <part name="SUPPLY51" library="_power_symbols" deviceset="AGND" device=""/>
@@
 <part name="SERVO_RING" library="_motors" deviceset="SERVO" device="_HK15298B_PTH_VERT_MALE_2.54MM" package3d_urn="urn:adsk.eagle:package:4781732/1" value="HK15298B"/>
 <part name="SERVO_PINKY" library="_motors" deviceset="SERVO" device="_HK15298B_PTH_VERT_MALE_2.54MM" package3d_urn="urn:adsk.eagle:package:4781732/1" value="HK15298B"/>
-<part name="C27" library="_capacitors" deviceset="1000UF-POLARIZED" device="_PTH_16V-20%" package3d_urn="urn:adsk.eagle:package:3036236/2" value="1000uF/16V"/>
+<part name="C27" library="_capacitors" deviceset="1000UF-POLARIZED" device="_PTH_16V-20%_D8-LS3.5-H20" package3d_urn="urn:adsk.eagle:package:9488079/1" value="1000uF/16V"/>
 <part name="J1" library="_connectors" deviceset="POWER_JACK-BARREL_ID2.1MM-OD5.5MM" device="_PTH_ID2.1MM-OD5.5MM" package3d_urn="urn:adsk.eagle:package:3034525/4" value="5A/28V"/>
-<part name="C9" library="_capacitors" deviceset="100UF-POLARIZED" device="_SMD_25V-20%_DIA5-LS2-H11" package3d_urn="urn:adsk.eagle:package:5948134/2" value="100uF/25V"/>
-<part name="C11" library="_capacitors" deviceset="100UF-POLARIZED" device="_SMD_25V-20%_DIA5-LS2-H11" package3d_urn="urn:adsk.eagle:package:5948134/2" value="100uF/25V"/>
-<part name="C13" library="_capacitors" deviceset="100UF-POLARIZED" device="_SMD_25V-20%_DIA5-LS2-H11" package3d_urn="urn:adsk.eagle:package:5948134/2" value="100uF/25V"/>
-<part name="C15" library="_capacitors" deviceset="100UF-POLARIZED" device="_SMD_25V-20%_DIA5-LS2-H11" package3d_urn="urn:adsk.eagle:package:5948134/2" value="100uF/25V"/>
-<part name="C17" library="_capacitors" deviceset="100UF-POLARIZED" device="_SMD_25V-20%_DIA5-LS2-H11" package3d_urn="urn:adsk.eagle:package:5948134/2" value="100uF/25V"/>
+<part name="C9" library="_capacitors" deviceset="100UF-POLARIZED" device="_PTH_25V-20%_D5-LS2-H11" package3d_urn="urn:adsk.eagle:package:9488069/1" value="100uF/25V"/>
+<part name="C11" library="_capacitors" deviceset="100UF-POLARIZED" device="_PTH_25V-20%_D5-LS2-H11" package3d_urn="urn:adsk.eagle:package:9488069/1" value="100uF/25V"/>
+<part name="C13" library="_capacitors" deviceset="100UF-POLARIZED" device="_PTH_25V-20%_D5-LS2-H11" package3d_urn="urn:adsk.eagle:package:9488069/1" value="100uF/25V"/>
+<part name="C15" library="_capacitors" deviceset="100UF-POLARIZED" device="_PTH_25V-20%_D5-LS2-H11" package3d_urn="urn:adsk.eagle:package:9488069/1" value="100uF/25V"/>
+<part name="C17" library="_capacitors" deviceset="100UF-POLARIZED" device="_PTH_25V-20%_D5-LS2-H11" package3d_urn="urn:adsk.eagle:package:9488069/1" value="100uF/25V"/>
 <part name="SUPPLY13" library="_power_symbols" deviceset="3.3V" device=""/>
 <part name="SUPPLY19" library="_power_symbols" deviceset="3.3V" device=""/>
@@
 <part name="D2" library="_discrete_semiconductors" deviceset="GENERAL-PURPOSE" device="_SMD_GP_1A-50V" package3d_urn="urn:adsk.eagle:package:2939213/1" value="1A/50V"/>
 <part name="SUPPLY22" library="_power_symbols" deviceset="A1.8V" device=""/>
+<part name="SW1" library="_switches" deviceset="SWITCH_SPDT" device="_VERT_PTH_5A-28V_13L-7W_" package3d_urn="urn:adsk.eagle:package:3033359/8" value="5A/28V"/>
 </parts>
 <sheets>
@@
 <instance part="GND124" gate="GND" x="157.48" y="152.4" smashed="yes"/>
 <instance part="NGND1" gate="G$1" x="142.24" y="152.4" smashed="yes"/>
-<instance part="SW1" gate="G$1" x="182.88" y="182.88" smashed="yes" rot="R180">
-<attribute name="NAME" x="181.61" y="179.832" size="1.27" layer="95" font="vector" ratio="10" rot="R180" align="bottom-center"/>
-<attribute name="VALUE" x="181.61" y="186.182" size="0.635" layer="96" font="vector" ratio="10" rot="R180" align="top-center"/>
-</instance>
 <instance part="GND125" gate="GND" x="254" y="162.56" smashed="yes"/>
 <instance part="D7" gate="G$1" x="252.73" y="149.86" smashed="yes" rot="R90">
@@
 </instance>
 <instance part="SUPPLY22" gate="G$1" x="205.74" y="330.2" smashed="yes"/>
+<instance part="SW1" gate="G$1" x="182.88" y="182.88" smashed="yes" rot="R180">
+<attribute name="NAME" x="181.61" y="179.832" size="1.27" layer="95" font="vector" ratio="10" rot="R180" align="bottom-center"/>
+<attribute name="VALUE" x="181.61" y="186.182" size="0.635" layer="96" font="vector" ratio="10" rot="R180" align="top-center"/>
+</instance>
 </instances>
 <busses>
@@
 <wire x1="154.94" y1="180.34" x2="172.72" y2="180.34" width="0.1524" layer="91"/>
 <pinref part="J1" gate="G$1" pin="PWR"/>
-<pinref part="SW1" gate="G$1" pin="S1"/>
 <wire x1="177.8" y1="180.34" x2="172.72" y2="180.34" width="0.1524" layer="91"/>
 <junction x="172.72" y="180.34"/>
 <pinref part="LIPO1" gate="G$1" pin="+"/>
+<pinref part="SW1" gate="G$1" pin="S1"/>
 </segment>
 </net>
@@
 <pinref part="C27" gate="G$1" pin="A"/>
 <pinref part="SUPPLY5" gate="G$1" pin="VBAT"/>
-<pinref part="SW1" gate="G$1" pin="P"/>
 <wire x1="185.42" y1="182.88" x2="193.04" y2="182.88" width="0.1524" layer="91"/>
 <pinref part="D2" gate="G$1" pin="K"/>
@@
 <wire x1="241.3" y1="190.5" x2="241.3" y2="182.88" width="0.1524" layer="91"/>
 <junction x="241.3" y="182.88"/>
-</segment>
-</net>
+<pinref part="SW1" gate="G$1" pin="P"/>
+</segment>
+</net>

Commit message: Lots of changes.  But rip.
Parts:
- C61: value 22pF/100V -> 22pF/100V/0402
Changed lines of the file:
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@@
 <part name="GND97" library="_power_symbols" deviceset="AGND" device=""/>
 <part name="B1" library="_radio_frequency" deviceset="BALUN" device="_SMD-0805_UNBAL/BAL-50/100" package3d_urn="urn:adsk.eagle:package:2933573/1" value="50/100"/>
-<part name="C61" library="_capacitors" deviceset="22PF" device="_CER_SMD-0402-100V-5%" package3d_urn="urn:adsk.eagle:package:2886515/1" value="22pF/100V"/>
+<part name="C61" library="_capacitors" deviceset="22PF" device="_CER_SMD-0402-100V-5%" package3d_urn="urn:adsk.eagle:package:2886515/1" value="22pF/100V/0402"/>
 <part name="C62" library="_capacitors" deviceset="0.75PF" device="_CER_SMD-0402_50V-33%" package3d_urn="urn:adsk.eagle:package:2886515/1" value="0.75pF/50V"/>
 <part name="A6" library="_radio_frequency" deviceset="ANTENNA" device="_SMD_CHP-2.45GHZ-0.5DBI-3W" package3d_urn="urn:adsk.eagle:package:2933495/1" value="2.45GHz"/>
@@
 </instance>
 <instance part="A6" gate="G$1" x="167.64" y="284.48" smashed="yes" rot="MR0">
-<attribute name="VALUE" x="167.132" y="283.972" size="1.27" layer="96" font="vector" ratio="10" rot="MR0" align="top-left"/>
+<attribute name="VALUE" x="167.132" y="283.972" size="0.635" layer="96" font="vector" ratio="10" rot="MR0" align="top-left"/>
 <attribute name="NAME" x="167.132" y="284.988" size="1.27" layer="95" font="vector" ratio="10" rot="MR0"/>
 </instance>

Commit message: Everything fucking works (have not tested ET driver extensively yet though)
Connections:
- net FSR_INDEX: now also FSR_INDEX.-; no longer FSR_RING.-
- net FSR_PINKY: now also FSR_PINKY.-; no longer FSR_THUMB.-
- net FSR_RING: now also FSR_RING.-; no longer FSR_INDEX.-
- net FSR_THUMB: now also FSR_THUMB.-; no longer FSR_PINKY.-
Other:
- moved on the sheet: FSR_INDEX, FSR_PINKY, FSR_RING, FSR_THUMB
Changed lines of the file:
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@@
 <part name="C98" library="_capacitors" deviceset="0.1UF" device="_SMD-0402_50V-10%" package3d_urn="urn:adsk.eagle:package:2886515/1" value="0.1uF/50V"/>
 <part name="VREG-MCU" library="_ic_power" deviceset="VREG_TPS768XX_ULDO_FAST-TRANSIENT" device="_TPS76833QDR_1A-3.3V" package3d_urn="urn:adsk.eagle:package:2899754/1" value="TPS76833QDR 1A/3.3V"/>
+<part name="FSR_THUMB" library="_sensors" deviceset="FORCE-SENSITIVE-RESISTOR_SENSOR" device="_FSR-5MM_0530470210_VERT-MALE_PITCH-1.25MM" package3d_urn="urn:adsk.eagle:package:2973718/2" value="10K"/>
+<part name="FSR_INDEX" library="_sensors" deviceset="FORCE-SENSITIVE-RESISTOR_SENSOR" device="_FSR-5MM_0530470210_VERT-MALE_PITCH-1.25MM" package3d_urn="urn:adsk.eagle:package:2973718/2" value="10K"/>
+<part name="FSR_MIDDLE" library="_sensors" deviceset="FORCE-SENSITIVE-RESISTOR_SENSOR" device="_FSR-5MM_0530470210_VERT-MALE_PITCH-1.25MM" package3d_urn="urn:adsk.eagle:package:2973718/2" value="10K"/>
+<part name="FSR_RING" library="_sensors" deviceset="FORCE-SENSITIVE-RESISTOR_SENSOR" device="_FSR-5MM_0530470210_VERT-MALE_PITCH-1.25MM" package3d_urn="urn:adsk.eagle:package:2973718/2" value="10K"/>
 <part name="FSR_PINKY" library="_sensors" deviceset="FORCE-SENSITIVE-RESISTOR_SENSOR" device="_FSR-5MM_0530470210_VERT-MALE_PITCH-1.25MM" package3d_urn="urn:adsk.eagle:package:2973718/2" value="10K"/>
-<part name="FSR_RING" library="_sensors" deviceset="FORCE-SENSITIVE-RESISTOR_SENSOR" device="_FSR-5MM_0530470210_VERT-MALE_PITCH-1.25MM" package3d_urn="urn:adsk.eagle:package:2973718/2" value="10K"/>
-<part name="FSR_MIDDLE" library="_sensors" deviceset="FORCE-SENSITIVE-RESISTOR_SENSOR" device="_FSR-5MM_0530470210_VERT-MALE_PITCH-1.25MM" package3d_urn="urn:adsk.eagle:package:2973718/2" value="10K"/>
-<part name="FSR_INDEX" library="_sensors" deviceset="FORCE-SENSITIVE-RESISTOR_SENSOR" device="_FSR-5MM_0530470210_VERT-MALE_PITCH-1.25MM" package3d_urn="urn:adsk.eagle:package:2973718/2" value="10K"/>
-<part name="FSR_THUMB" library="_sensors" deviceset="FORCE-SENSITIVE-RESISTOR_SENSOR" device="_FSR-5MM_0530470210_VERT-MALE_PITCH-1.25MM" package3d_urn="urn:adsk.eagle:package:2973718/2" value="10K"/>
 <part name="SUPPLY11" library="_power_symbols" deviceset="5V" device=""/>
 <part name="SUPPLY12" library="_power_symbols" deviceset="5V" device=""/>
@@
 <attribute name="VALUE" x="254" y="185.166" size="0.635" layer="95" font="vector" ratio="10" align="top-center"/>
 </instance>
-<instance part="FSR_PINKY" gate="G$1" x="340.36" y="218.44" smashed="yes">
+<instance part="FSR_THUMB" gate="G$1" x="340.36" y="218.44" smashed="yes">
 <attribute name="NAME" x="341.63" y="221.488" size="1.27" layer="95" font="vector" ratio="10" align="bottom-right"/>
 <attribute name="VALUE" x="341.63" y="213.106" size="0.635" layer="96" font="vector" ratio="10" align="top-right"/>
 </instance>
-<instance part="FSR_RING" gate="G$1" x="340.36" y="185.42" smashed="yes">
+<instance part="FSR_INDEX" gate="G$1" x="340.36" y="185.42" smashed="yes">
 <attribute name="NAME" x="341.63" y="188.468" size="1.27" layer="95" font="vector" ratio="10" align="bottom-right"/>
 <attribute name="VALUE" x="341.63" y="180.086" size="0.635" layer="96" font="vector" ratio="10" align="top-right"/>
@@
 <attribute name="VALUE" x="341.63" y="147.066" size="0.635" layer="96" font="vector" ratio="10" align="top-right"/>
 </instance>
-<instance part="FSR_INDEX" gate="G$1" x="340.36" y="119.38" smashed="yes">
+<instance part="FSR_RING" gate="G$1" x="340.36" y="119.38" smashed="yes">
 <attribute name="NAME" x="341.63" y="122.428" size="1.27" layer="95" font="vector" ratio="10" align="bottom-right"/>
 <attribute name="VALUE" x="341.63" y="114.046" size="0.635" layer="96" font="vector" ratio="10" align="top-right"/>
 </instance>
-<instance part="FSR_THUMB" gate="G$1" x="340.36" y="86.36" smashed="yes">
+<instance part="FSR_PINKY" gate="G$1" x="340.36" y="86.36" smashed="yes">
 <attribute name="NAME" x="341.63" y="89.408" size="1.27" layer="95" font="vector" ratio="10" align="bottom-right"/>
 <attribute name="VALUE" x="341.63" y="81.026" size="0.635" layer="96" font="vector" ratio="10" align="top-right"/>
@@
 <wire x1="347.98" y1="83.82" x2="345.44" y2="83.82" width="0.1524" layer="91"/>
 <junction x="345.44" y="83.82"/>
-<pinref part="FSR_THUMB" gate="G$1" pin="-"/>
+<pinref part="FSR_PINKY" gate="G$1" pin="-"/>
 </segment>
 <segment>
@@
 <wire x1="347.98" y1="116.84" x2="345.44" y2="116.84" width="0.1524" layer="91"/>
 <junction x="345.44" y="116.84"/>
-<pinref part="FSR_INDEX" gate="G$1" pin="-"/>
+<pinref part="FSR_RING" gate="G$1" pin="-"/>
 </segment>
 <segment>
@@
 <wire x1="347.98" y1="182.88" x2="345.44" y2="182.88" width="0.1524" layer="91"/>
 <junction x="345.44" y="182.88"/>
-<pinref part="FSR_RING" gate="G$1" pin="-"/>
+<pinref part="FSR_INDEX" gate="G$1" pin="-"/>
 </segment>
 <segment>
@@
 <wire x1="347.98" y1="215.9" x2="345.44" y2="215.9" width="0.1524" layer="91"/>
 <junction x="345.44" y="215.9"/>
-<pinref part="FSR_PINKY" gate="G$1" pin="-"/>
+<pinref part="FSR_THUMB" gate="G$1" pin="-"/>
 </segment>
 <segment>
@@
 <wire x1="342.9" y1="218.44" x2="345.44" y2="218.44" width="0.1524" layer="91"/>
 <wire x1="345.44" y1="218.44" x2="345.44" y2="220.98" width="0.1524" layer="91"/>
-<pinref part="FSR_PINKY" gate="G$1" pin="+"/>
+<pinref part="FSR_THUMB" gate="G$1" pin="+"/>
 <pinref part="SUPPLY1" gate="G$1" pin="VSENSOR"/>
 </segment>
@@
 <wire x1="342.9" y1="185.42" x2="345.44" y2="185.42" width="0.1524" layer="91"/>
 <wire x1="345.44" y1="185.42" x2="345.44" y2="187.96" width="0.1524" layer="91"/>
-<pinref part="FSR_RING" gate="G$1" pin="+"/>
+<pinref part="FSR_INDEX" gate="G$1" pin="+"/>
 <pinref part="SUPPLY3" gate="G$1" pin="VSENSOR"/>
 </segment>
@@
 <wire x1="342.9" y1="119.38" x2="345.44" y2="119.38" width="0.1524" layer="91"/>
 <wire x1="345.44" y1="119.38" x2="345.44" y2="121.92" width="0.1524" layer="91"/>
-<pinref part="FSR_INDEX" gate="G$1" pin="+"/>
+<pinref part="FSR_RING" gate="G$1" pin="+"/>
 <pinref part="SUPPLY38" gate="G$1" pin="VSENSOR"/>
 </segment>
@@
 <wire x1="342.9" y1="86.36" x2="345.44" y2="86.36" width="0.1524" layer="91"/>
 <wire x1="345.44" y1="86.36" x2="345.44" y2="88.9" width="0.1524" layer="91"/>
-<pinref part="FSR_THUMB" gate="G$1" pin="+"/>
+<pinref part="FSR_PINKY" gate="G$1" pin="+"/>
 <pinref part="SUPPLY44" gate="G$1" pin="VSENSOR"/>
 </segment>
