File: ecad/touch_glove/touch_glove.brd (EAGLE design)
At the start: 80 x 38.4 mm, 143 parts, among them J9 PTH VERT MALE, Q1 MCH3474 4A/30V, Q2 MCH3474 4A/30V, Q3 MCH3474 4A/30V, Q4 MCH3474 4A/30V, Q5 MCH3474 4A/30V, Q6 MCH3474 4A/30V, SW1 4A/28V

Commit message: Lots of changes.  But rip.
Changed lines of the file:
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@@
 <layers>
 <layer number="1" name="Top" color="4" fill="1" visible="yes" active="yes"/>
-<layer number="2" name="Route2" color="4" fill="6" visible="yes" active="yes"/>
+<layer number="2" name="Route2" color="4" fill="6" visible="no" active="yes"/>
 <layer number="3" name="Route3" color="4" fill="3" visible="no" active="no"/>
 <layer number="4" name="Route4" color="1" fill="4" visible="no" active="no"/>
@@
 <layer number="13" name="Route13" color="4" fill="5" visible="no" active="no"/>
 <layer number="14" name="Route14" color="1" fill="6" visible="no" active="no"/>
-<layer number="15" name="Route15" color="1" fill="6" visible="yes" active="yes"/>
+<layer number="15" name="Route15" color="1" fill="6" visible="no" active="yes"/>
 <layer number="16" name="Bottom" color="1" fill="1" visible="yes" active="yes"/>
 <layer number="17" name="Pads" color="2" fill="1" visible="yes" active="yes"/>
@@
 <layer number="21" name="tPlace" color="7" fill="1" visible="yes" active="yes"/>
 <layer number="22" name="bPlace" color="7" fill="1" visible="yes" active="yes"/>
-<layer number="23" name="tOrigins" color="15" fill="1" visible="no" active="yes"/>
-<layer number="24" name="bOrigins" color="15" fill="1" visible="no" active="yes"/>
-<layer number="25" name="tNames" color="7" fill="1" visible="no" active="yes"/>
-<layer number="26" name="bNames" color="7" fill="1" visible="no" active="yes"/>
-<layer number="27" name="tValues" color="7" fill="1" visible="no" active="yes"/>
+<layer number="23" name="tOrigins" color="15" fill="1" visible="yes" active="yes"/>
+<layer number="24" name="bOrigins" color="15" fill="1" visible="yes" active="yes"/>
+<layer number="25" name="tNames" color="7" fill="1" visible="yes" active="yes"/>
+<layer number="26" name="bNames" color="7" fill="1" visible="yes" active="yes"/>
+<layer number="27" name="tValues" color="7" fill="1" visible="yes" active="yes"/>
 <layer number="28" name="bValues" color="7" fill="1" visible="no" active="yes"/>
 <layer number="29" name="tStop" color="7" fill="3" visible="no" active="yes"/>
@@
 <hole x="38.3" y="26.5" drill="2"/>
 <hole x="-38.5" y="10.5" drill="2"/>
+<text x="1.4" y="1" size="1" layer="21" font="vector" ratio="20">Transmission of Touch VR</text>
+<text x="28.4" y="1" size="0.7" layer="21" font="vector" ratio="20">Touch Glove     Rev 3</text>
 </plain>
 <attributes>
@@
 <attribute name="MPN" value="GRM155C80J106ME11D" x="-18" y="13.6" size="1.778" layer="27" display="off"/>
 <attribute name="NAME" x="-18" y="14.3" size="0.5" layer="25" font="vector" ratio="10" align="bottom-center"/>
-<attribute name="VALUE" x="-18" y="12.9" size="0.5" layer="27" font="vector" ratio="10" align="top-center"/>
+<attribute name="VALUE" x="-18" y="12.9" size="0.25" layer="27" font="vector" ratio="10" align="top-center"/>
 </element>
 <element name="C9" library="_capacitors" package="CAPC1005X55_SMD-0402" package3d_urn="urn:adsk.eagle:package:2886515/1" value="0.1uF/50V" x="-18" y="14.9" smashed="yes">
@@
 <attribute name="MPN" value="C1005X7R1H104K050BE" x="-18" y="14.9" size="1.778" layer="27" display="off"/>
 <attribute name="NAME" x="-18" y="15.6" size="0.5" layer="25" font="vector" ratio="10" align="bottom-center"/>
-<attribute name="VALUE" x="-18" y="14.2" size="0.5" layer="27" font="vector" ratio="10" align="top-center"/>
+<attribute name="VALUE" x="-18" y="14.2" size="0.25" layer="27" font="vector" ratio="10" align="top-center"/>
 </element>
 <element name="C18" library="_capacitors" package="CAPCP3216X160" package3d_urn="urn:adsk.eagle:package:6906990/1" value="100uF/10V" x="-7.9" y="17.4" smashed="yes" rot="R180">
@@
 <attribute name="MPN_CRIMP" value="0500798000" x="-18.9" y="6.7" size="1.778" layer="27" font="vector" rot="R180" display="off"/>
 <attribute name="NAME" x="-18.94" y="4.42" size="0.5" layer="25" font="vector" ratio="10" align="top-center"/>
-<attribute name="VALUE" x="-16.36" y="9.24" size="1.27" layer="27" font="vector" ratio="10" rot="R180"/>
+<attribute name="VALUE" x="-18.46" y="5.84" size="0.25" layer="27" font="vector" ratio="10" rot="R180"/>
 </element>
 <element name="BR_ANALOG" library="_power_symbols" package="NET_BRIDGE" value="NET_BRIDGE" x="-19.9" y="5" smashed="yes" rot="MR270"/>

Commit message: Everything fucking works (have not tested ET driver extensively yet though)
Parts:
- C36: value 22pF/100V -> 22pF/100V/0402
Changed lines of the file:
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@@
 </layers>
 <board>
-<fusionsync huburn="a.cGVyc29uYWw6dWUyOTIwMzJm" projecturn="a.cGVyc29uYWw6dWUyOTIwMzJmIzIwMTgwNTE1MTMyMDQwMDA2" f3durn="urn:adsk.wipprod:dm.lineage:BV8_dkhaR6yVWje6GJc8ag" pcbguid="eeba273b-519e-40e6-aef7-dc52009e201f" lastpulledtime="" lastsyncedchangeguid="37155c65-f2cb-0758-bd04-201c3b8eaef8"/>
+<fusionsync huburn="a.cGVyc29uYWw6dWUyOTIwMzJm" projecturn="a.cGVyc29uYWw6dWUyOTIwMzJmIzIwMTgwNTE1MTMyMDQwMDA2" f3durn="urn:adsk.wipprod:dm.lineage:BV8_dkhaR6yVWje6GJc8ag" pcbguid="eeba273b-519e-40e6-aef7-dc52009e201f" lastpulledtime="" lastsyncedchangeguid="2c0f9fad-1720-cee9-cd53-b6f6876c3a39"/>
 <plain>
 <wire x1="38.6992" y1="38.44" x2="-38.6992" y2="38.44" width="0" layer="20"/>
@@
 <attribute name="VALUE" x="12.3" y="15.1" size="0.5" layer="27" font="vector" ratio="10" rot="R270" align="top-center"/>
 </element>
-<element name="C36" library="_capacitors" package="CAPC1005X55_SMD-0402" package3d_urn="urn:adsk.eagle:package:2886515/1" value="22pF/100V" x="27" y="9.9" smashed="yes">
-<attribute name="DATASHEET" value="http://ds.yuden.co.jp/TYCOMPAS/ut/detail.do?productNo=HMK105CG220JV-F&amp;fileName=HMK105CG220JV-F_SS&amp;mode=specSheetDownload" x="27" y="9.9" size="1.778" layer="27" display="off"/>
+<element name="C36" library="_capacitors" package="CAPC1005X55_SMD-0402" package3d_urn="urn:adsk.eagle:package:2886515/1" value="22pF/100V/0402" x="27" y="9.9" smashed="yes">
+<attribute name="DATASHEET" value="http://www.vishay.com/docs/45071/vjhifreq.pdf" x="27" y="9.9" size="1.778" layer="27" display="off"/>
 <attribute name="DIST" value="Digikey" x="27" y="9.9" size="1.778" layer="27" display="off"/>
-<attribute name="DISTLINK" value="https://www.digikey.com/products/en?keywords=587-5004-1-ND" x="27" y="9.9" size="1.778" layer="27" display="off"/>
-<attribute name="DISTPN" value="587-5004-1-ND" x="27" y="9.9" size="1.778" layer="27" display="off"/>
-<attribute name="MFR" value="Taiyo Yuden" x="27" y="9.9" size="1.778" layer="27" display="off"/>
-<attribute name="MPN" value="HMK105CG220JV-F" x="27" y="9.9" size="1.778" layer="27" display="off"/>
+<attribute name="DISTLINK" value="https://www.digikey.com/products/en?keywords=720-1286-1-ND" x="27" y="9.9" size="1.778" layer="27" display="off"/>
+<attribute name="DISTPN" value="720-1286-1-ND" x="27" y="9.9" size="1.778" layer="27" display="off"/>
+<attribute name="MFR" value="Vishay Vitramon" x="27" y="9.9" size="1.778" layer="27" display="off"/>
+<attribute name="MPN" value="VJ0402D220JXBAJ" x="27" y="9.9" size="1.778" layer="27" display="off"/>
 <attribute name="NAME" x="27" y="10.6" size="0.5" layer="25" font="vector" ratio="10" align="bottom-center"/>
-<attribute name="VALUE" x="27" y="9.2" size="0.5" layer="27" font="vector" ratio="10" align="top-center"/>
+<attribute name="VALUE" value="22pF/100V/0402" x="27" y="9.2" size="0.5" layer="27" font="vector" ratio="10" align="top-center"/>
 </element>
 <element name="C35" library="_capacitors" package="CAPC1005X55_SMD-0402" package3d_urn="urn:adsk.eagle:package:2886515/1" value="0.75pF/50V" x="27" y="8.6" smashed="yes">
